Commit message: some updates to fix issues. Not completely done but gives better starting point

File: src/arm_ws/src/arm/urdf/robot_arm.urdf (robot description, URDF)
Before this commit: robot robot_arm, 4 links, 3 joints
Links:
- link base_link: geometry collision box size=0.1 0.1 0.1; visual box size=0.1 0.1 0.1
- link end_effector: mass None -> 0.1
- link link1: mass None -> 1
- link link2: mass None -> 1
Joints:
- joint joint1: limit lower=-1.57 upper=1.57 -> lower=-1.57 upper=1.57 effort=1000 velocity=10
- joint joint2: limit lower=-1.57 upper=1.57 -> lower=-1.57 upper=1.57 effort=1000 velocity=10
- joint joint3: limit lower=-1.57 upper=1.57 -> lower=-1.57 upper=1.57 effort=1000 velocity=10
