Commit message: added wheels to urdf

File: src/rover_description/src/description.urdf (robot description, URDF)
Before this commit: robot uiowa_rover, 2 links, 1 joints
Links:
- added link back_l_wheel; collision cylinder length=${wheel_width} radius=${wheel_diameter/2}; visual cylinder length=${wheel_width} radius=${wheel_diameter/2}
- added link back_r_wheel; collision cylinder length=${wheel_width} radius=${wheel_diameter/2}; visual cylinder length=${wheel_width} radius=${wheel_diameter/2}
- added link chassis; collision box size=${arm_platform_length} ${arm_platform_width} ${arm_platform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; collision box size=${chassis_length} ${chassis_width} ${chassis_height}
- added link front_l_wheel; collision cylinder length=${wheel_width} radius=${wheel_diameter/2}; visual cylinder length=${wheel_width} radius=${wheel_diameter/2}
- added link front_r_wheel; collision cylinder length=${wheel_width} radius=${wheel_diameter/2}; visual cylinder length=${wheel_width} radius=${wheel_diameter/2}
- added link mid_l_wheel; collision cylinder length=${wheel_width} radius=${wheel_diameter/2}; visual cylinder length=${wheel_width} radius=${wheel_diameter/2}
- added link mid_r_wheel; collision cylinder length=${wheel_width} radius=${wheel_diameter/2}; visual cylinder length=${wheel_width} radius=${wheel_diameter/2}
- link base_link: geometry 
Joints:
- added joint back_l_wheel_joint: type continuous, parent chassis, child back_l_wheel, origin xyz=${chassis_length/2.5-wheel_spacing} ${wheel_distance_side} ${-suspension_height-(chassis_height/2)} rpy=${pi/2} 0 0, axis 0 0 1
- added joint back_r_wheel_joint: type continuous, parent chassis, child back_r_wheel, origin xyz=${chassis_length/2.5-wheel_spacing} ${-wheel_distance_side} ${-suspension_height-(chassis_height/2)} rpy=${pi/2} 0 0, axis 0 0 1
- added joint chasiss_joint: type fixed, parent base_link, child chassis, origin xyz=0 0 0 rpy=0 0 0
- added joint front_l_wheel_joint: type continuous, parent chassis, child front_l_wheel, origin xyz=${chassis_length/2.5+wheel_spacing} ${wheel_distance_side} ${-suspension_height-(chassis_height/2)} rpy=${pi/2} 0 0, axis 0 0 1
- added joint front_r_wheel_joint: type continuous, parent chassis, child front_r_wheel, origin xyz=${chassis_length/2.5+wheel_spacing} ${-wheel_distance_side} ${-suspension_height-(chassis_height/2)} rpy=${pi/2} 0 0, axis 0 0 1
- added joint mid_l_wheel_joint: type continuous, parent chassis, child mid_l_wheel, origin xyz=${chassis_length/2.5} ${wheel_distance_side} ${-suspension_height-(chassis_height/2)} rpy=${pi/2} 0 0, axis 0 0 1
- added joint mid_r_wheel_joint: type continuous, parent chassis, child mid_r_wheel, origin xyz=${chassis_length/2.5} ${-wheel_distance_side} ${-suspension_height-(chassis_height/2)} rpy=${pi/2} 0 0, axis 0 0 1
- joint base_joint: origin xyz=0.0 0.0 0.0 rpy=0 0 0 -> xyz=0.0 0.0 ${-0.3-chassis_height/2} rpy=0 0 0
