Commit message: gazebo camera support

File: src/uirover_description/urdf/uirover.urdf (robot description, URDF)
Before this commit: robot uirover, 14 links, 13 joints
Links:
- added link demo_camera, mass 0.1; collision cylinder length=0.01 radius=0.01; visual cylinder length=0.01 radius=0.01
Joints:
- added joint front_camera_joint: type fixed, parent base_link, child demo_camera, origin xyz=1.0 0.0 0.0 rpy=0.0 0.0 0.0

File: src/uirover_description/urdf/uirover.urdf.xacro (robot description, xacro)
@@ -1,6 +1,8 @@
 <?xml version="1.0"?>
 <robot name="uirover" xmlns:xacro="http://www.ros.org/wiki/xacro">
-    <xacro:include filename="$(find uirover_description)/urdf_components/physical_description.urdf.xacro"/>
-    <xacro:include filename="$(find uirover_description)/urdf_components/sensors.urdf.xacro"/>
-    <xacro:include filename="$(find uirover_description)/urdf_components/ros2_control.urdf.xacro"/>
+    <xacro:include filename="$(find uirover_description)/xacro/physical_description.urdf.xacro"/>
+    <xacro:include filename="$(find uirover_description)/xacro/sensors.urdf.xacro"/>
+    <xacro:include filename="$(find uirover_description)/xacro/ros2_control.urdf.xacro"/>
+    <xacro:uirover_ros2_control use_gazebo="false"/>
+    <xacro:uirover_sensors use_gazebo="false"/>
 </robot>

File: src/uirover_description/urdf/uirover_sim.urdf (robot description, URDF)
Before this commit: robot uirover, 14 links, 13 joints
Links:
- added link demo_camera, mass 0.1; collision cylinder length=0.01 radius=0.01; visual cylinder length=0.01 radius=0.01
Joints:
- added joint front_camera_joint: type fixed, parent base_link, child demo_camera, origin xyz=1.0 0.0 0.0 rpy=0.0 0.0 0.0

File: src/uirover_description/urdf/uirover_sim.urdf.xacro (robot description, xacro)
@@ -1,7 +1,9 @@
 <?xml version="1.0"?>
 <robot name="uirover" xmlns:xacro="http://www.ros.org/wiki/xacro">
-    <xacro:include filename="$(find uirover_description)/urdf_components/physical_description.urdf.xacro"/>
-    <xacro:include filename="$(find uirover_description)/urdf_components/sensors.urdf.xacro"/>
-    <xacro:include filename="$(find uirover_description)/urdf_components/ros2_control.urdf.xacro"/>
-    <xacro:include filename="$(find uirover_description)/urdf_components/gazebo.urdf.xacro"/>
+    <xacro:include filename="$(find uirover_description)/xacro/gazebo.urdf.xacro"/>
+    <xacro:include filename="$(find uirover_description)/xacro/physical_description.urdf.xacro"/>
+    <xacro:include filename="$(find uirover_description)/xacro/sensors.urdf.xacro"/>
+    <xacro:include filename="$(find uirover_description)/xacro/ros2_control.urdf.xacro"/>
+    <xacro:uirover_ros2_control use_gazebo="true"/>
+    <xacro:uirover_sensors use_gazebo="true"/>
 </robot>

File: src/uirover_description/xacro/physical_description.urdf.xacro (robot description, xacro)
@@ -2,5 +2,5 @@
 <robot name="uirover" xmlns:xacro="http://www.ros.org/wiki/xacro">
   <!-- IMPORTS -->
-  <xacro:include filename="$(find uirover_description)/xacro/macros.xacro" />
+  <xacro:include filename="$(find uirover_description)/xacro/utility_macros.xacro" />
   <xacro:include filename="$(find uirover_description)/xacro/properties.xacro" />
   <!-- BASE LINK -->

File: src/uirover_description/xacro/ros2_control.urdf.xacro (robot description, xacro)
@@ -11,10 +11,10 @@
                     <plugin>gz_ros2_control/GazeboSimSystem</plugin>
                 </xacro:if>
-                <xacro:unless value="${use_gazebo}">
+                <!-- <xacro:unless value="${use_gazebo}">
                     <plugin>uirover_hardware/RRBotSystemPositionOnlyHardware</plugin>
                     <param name="example_param_hw_start_duration_sec">0</param>
                     <param name="example_param_hw_stop_duration_sec">3.0</param>
                     <param name="example_param_hw_slowdown">100</param>
-                </xacro:unless>
+                </xacro:unless> -->
             </hardware>
         </ros2_control>

File: src/uirover_description/xacro/utility_macros.xacro (robot description, xacro)
@@ -1,5 +1,5 @@
 <?xml version="1.0" encoding="UTF-8"?>
 <robot name="uiowa_rover" xmlns:xacro="http://ros.org/wiki/xacro">
-  <!-- INERTIA -->
+  <!-- BOX INERTIA -->
   <xacro:macro name="box_inertia_tensor" params="mass len_x len_y len_z">
     <inertial>
@@ -10,4 +10,5 @@
     </inertial>
   </xacro:macro>
+  <!-- CYLINDER INERTIA -->
   <xacro:macro name="cylinder_inertia_tensor" params="mass radius length">
     <inertial>
@@ -18,5 +19,5 @@
     </inertial>
   </xacro:macro>
-  <!-- BOX -->
+  <!-- COLLIDABLE BOX -->
   <xacro:macro name="box" params="name x y z mass">
     <link name="${name}">

Commit message: upgrades

File: src/uirover_description/urdf/uirover.urdf (robot description, URDF)
Before this commit: robot uirover, 15 links, 14 joints
Links:
- link demo_camera: geometry collision cylinder length=0.01 radius=0.01; visual box size=0.005 0.03 0.03
Joints:
- joint front_camera_joint: origin xyz=1.0 0.0 0.0 rpy=0.0 0.0 0.0 -> xyz=0.0 0.2 0.8 rpy=0.0 0.5 0.0

File: src/uirover_description/urdf/uirover_sim.urdf (robot description, URDF)
Before this commit: robot uirover, 15 links, 14 joints
Links:
- link demo_camera: geometry collision cylinder length=0.01 radius=0.01; visual box size=0.005 0.03 0.03
Joints:
- joint front_camera_joint: origin xyz=1.0 0.0 0.0 rpy=0.0 0.0 0.0 -> xyz=0.0 0.2 0.8 rpy=0.0 0.5 0.0

File: src/uirover_description/xacro/sensors.urdf.xacro (robot description, xacro)
@@ -7,50 +7,10 @@
         <!-- =============================== -->
         <!-- ARDUCAM CAMERA -->
-        <xacro:macro name="arducam" params="name use_gazebo:=^|false">
-            <link name="${name}">
-                <visual>
-                    <geometry>
-                        <cylinder radius="0.01" length="0.01" />
-                    </geometry>
-                    <material name="Grey">
-                        <color rgba="0.7 0.7 0.7 1.0" />
-                    </material>
-                </visual>
-                <collision>
-                    <geometry>
-                        <cylinder radius="0.01" length="0.01" />
-                    </geometry>
-                </collision>
-                <xacro:cylinder_inertia_tensor mass="0.1" radius="0.01" length="0.01" />
-            </link>
-            <xacro:if value="${use_gazebo}">
-                <gazebo reference="${name}">
-                    <sensor name="boundingbox_camera" type="boundingbox_camera">
-                        <topic>demo_cam</topic>
-                        <camera>
-                            <box_type>2d</box_type>
-                            <horizontal_fov>1.047</horizontal_fov>
-                            <image>
-                                <width>800</width>
-                                <height>600</height>
-                            </image>
-                            <clip>
-                                <near>0.1</near>
-                                <far>10</far>
-                            </clip>
-                        </camera>
-                        <always_on>1</always_on>
-                        <update_rate>30</update_rate>
-                        <visualize>true</visualize>
-                    </sensor>
-                </gazebo>
-            </xacro:if>
-            <joint name="front_camera_joint" type="fixed">
-                <origin xyz="1.0 0.0 0.0" rpy="0.0 0.0 0.0" />
-                <parent link="base_link" />
-                <child link="${name}" />
-            </joint>
-        </xacro:macro>
         <xacro:arducam name="demo_camera" use_gazebo="true" />
+        <joint name="front_camera_joint" type="fixed">
+            <origin xyz="0.0 0.2 0.8" rpy="0.0 0.5 0.0" />
+            <parent link="base_link" />
+            <child link="demo_camera" />
+        </joint>
     </xacro:macro>
 </robot>

File: src/uirover_description/xacro/utility_macros.xacro (robot description, xacro)
@@ -90,3 +90,51 @@
     </joint>
   </xacro:macro>
+  <xacro:macro name="arducam" params="name use_gazebo:=^|false">
+    <link name="${name}">
+      <visual>
+        <origin xyz="0.0 0.0 0.0" rpy="0.0 ${pi/2} 0.0" />
+        <geometry>
+          <cylinder radius="0.01" length="0.01" />
+        </geometry>
+        <material name="Grey">
+          <color rgba="0.7 0.7 0.7 1.0" />
+        </material>
+      </visual>
+      <visual>
+        <origin xyz="-0.005 0.0 0.0" rpy="0.0 0.0 0.0" />
+        <geometry>
+          <box size="0.005 0.03 0.03" />
+        </geometry>
+      </visual>
+      <collision>
+        <geometry>
+          <cylinder radius="0.01" length="0.01" />
+        </geometry>
+      </collision>
+      <xacro:cylinder_inertia_tensor mass="0.1" radius="0.01" length="0.01" />
+    </link>
+    <xacro:if value="${use_gazebo}">
+      <gazebo reference="${name}">
+        <sensor name="boundingbox_camera" type="boundingbox_camera">
+          <topic>${name}</topic>
+          <camera>
+            <box_type>2d</box_type>
+            <!-- 110 deg FOV -->
+            <horizontal_fov>1.9198</horizontal_fov>
+            <image>
+              <width>800</width>
+              <height>600</height>
+            </image>
+            <clip>
+              <near>0.1</near>
+              <far>10</far>
+            </clip>
+          </camera>
+          <always_on>1</always_on>
+          <update_rate>30</update_rate>
+          <visualize>true</visualize>
+        </sensor>
+      </gazebo>
+    </xacro:if>
+  </xacro:macro>
 </robot>

Commit message: chassis plus suspension

File: src/uirover_description/urdf/uirover.urdf (robot description, URDF)
Before this commit: robot uirover, 15 links, 14 joints
Links:
- removed link arm_platform
- added link l_suspension; visual mesh filename=file:///home/ethan/Robotics/Rover/build/uirover_description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
- added link r_suspension; visual mesh filename=file:///home/ethan/Robotics/Rover/build/uirover_description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
- link chassis: mass 5 -> None; geometry visual mesh filename=file:///home/ethan/Robotics/Rover/build/uirover_description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
Joints:
- removed joint arm_platform_joint
- added joint l_suspension: type fixed, parent chassis, child l_suspension, origin xyz=0.35 0.28 0.1 rpy=0 0 0
- added joint r_suspension: type fixed, parent chassis, child r_suspension, origin xyz=0.35 -0.28 0.1 rpy=0 0 0

File: src/uirover_description/urdf/uirover_sim.urdf (robot description, URDF)
Before this commit: robot uirover, 15 links, 14 joints
Links:
- removed link arm_platform
- added link l_suspension; visual mesh filename=file:///home/ethan/Robotics/Rover/build/uirover_description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
- added link r_suspension; visual mesh filename=file:///home/ethan/Robotics/Rover/build/uirover_description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
- link chassis: mass 5 -> None; geometry visual mesh filename=file:///home/ethan/Robotics/Rover/build/uirover_description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
Joints:
- removed joint arm_platform_joint
- added joint l_suspension: type fixed, parent chassis, child l_suspension, origin xyz=0.35 0.28 0.1 rpy=0 0 0
- added joint r_suspension: type fixed, parent chassis, child r_suspension, origin xyz=0.35 -0.28 0.1 rpy=0 0 0

File: src/uirover_description/xacro/physical_description.urdf.xacro (robot description, xacro)
@@ -7,6 +7,12 @@
   <link name="base_link" />
   <!-- CHASSIS -->
-  <xacro:box name="chassis" x="${chassis_length}" y="${chassis_width}" z="${chassis_height}" mass="${5}" />
-  <xacro:box_inertia_tensor mass="${chassis_mass}" len_x="${chassis_length}" len_y="${chassis_width}" len_z="${chassis_height}" />
+  <link name="chassis">
+  <visual>
+    <origin xyz="0.0 0.21 0.0" rpy="${pi/2} 0.0 0.0"/>
+    <geometry>
+      <mesh filename="file://$(find uirover_description)/dae/chassis.dae"/>
+    </geometry>
+  </visual>
+  </link>
   <joint name="chassis_joint" type="fixed">
     <parent link="base_link" />
@@ -14,10 +20,31 @@
     <origin xyz="0 0 0" rpy="0 0 0" />
   </joint>
-  <!-- ARM PLATFORM -->
-  <xacro:box name="arm_platform" x="${arm_platform_length}" y="${arm_platform_width}" z="${arm_platform_height}" mass="${3}" />
-  <joint name="arm_platform_joint" type="fixed">
-    <parent link="base_link" />
-    <child link="arm_platform" />
-    <origin xyz="${chassis_length/2 + arm_platform_length/2} 0 ${-chassis_height/2 + arm_platform_height/2}" rpy="0 0 0" />
+  <!--L SUSPENSIONS-->
+  <link name="l_suspension">
+    <visual>
+    <origin xyz="-0.085 -0.02 -0.06" rpy="${pi/2} 0.0 0.0"/>
+    <geometry>
+      <mesh filename="file://$(find uirover_description)/dae/suspension.dae"/>
+    </geometry>
+  </visual>
+  </link>
+  <joint name="l_suspension" type="fixed">
+    <parent link="chassis" />
+    <child link="l_suspension" />
+    <origin xyz="0.35 0.28 0.1" rpy="0 0 0" />
+  </joint>
+  <!--R SUSPENSIONS-->
+  <link name="r_suspension">
+    <visual>
+    <origin xyz="-0.085 -0.02 -0.06" rpy="${pi/2} 0.0 0.0"/>
+    <geometry>
+      <mesh filename="file://$(find uirover_description)/dae/suspension.dae"/>
+    </geometry>
+  </visual>
+  </link>
+  <joint name="r_suspension" type="fixed">
+    <parent link="chassis" />
+    <child link="r_suspension" />
+    <origin xyz="0.35 -0.28 0.1" rpy="0 0 0" />
   </joint>
   <!-- SWIVEL JOINTS -->

Commit message: remove obsolete STL files and update URDF/Xacro paths for project relocation

File: src/uirover_description/urdf/uirover.urdf (robot description, URDF)
Before this commit: robot uirover, 16 links, 15 joints
Links:
- link chassis: geometry visual mesh filename=file:///home/ethan/Projects/Rover/build/uirover_description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
- link l_suspension: geometry visual mesh filename=file:///home/ethan/Projects/Rover/build/uirover_description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
- link r_suspension: geometry visual mesh filename=file:///home/ethan/Projects/Rover/build/uirover_description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

File: src/uirover_description/urdf/uirover_sim.urdf (robot description, URDF)
Before this commit: robot uirover, 16 links, 15 joints
Links:
- link chassis: geometry visual mesh filename=file:///home/ethan/Projects/Rover/build/uirover_description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
- link l_suspension: geometry visual mesh filename=file:///home/ethan/Projects/Rover/build/uirover_description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
- link r_suspension: geometry visual mesh filename=file:///home/ethan/Projects/Rover/build/uirover_description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

File: src/uirover_description/xacro/physical_description.urdf.xacro (robot description, xacro)
@@ -9,5 +9,5 @@
   <link name="chassis">
   <visual>
-    <origin xyz="0.0 0.21 0.0" rpy="${pi/2} 0.0 0.0"/>
+    <origin xyz="0.0 0.203 0.0" rpy="${pi/2} 0.0 0.0"/>
     <geometry>
       <mesh filename="file://$(find uirover_description)/dae/chassis.dae"/>
@@ -23,5 +23,5 @@
   <link name="l_suspension">
     <visual>
-    <origin xyz="-0.085 -0.02 -0.06" rpy="${pi/2} 0.0 0.0"/>
+      <origin xyz="0.085 0.02 -0.06" rpy="${pi/2} 0.0 ${pi}"/>
     <geometry>
       <mesh filename="file://$(find uirover_description)/dae/suspension.dae"/>
@@ -37,5 +37,5 @@
   <link name="r_suspension">
     <visual>
-    <origin xyz="-0.085 -0.02 -0.06" rpy="${pi/2} 0.0 0.0"/>
+      <origin xyz="0.085 0.02 -0.06" rpy="${pi/2} 0.0 ${pi}"/>
     <geometry>
       <mesh filename="file://$(find uirover_description)/dae/suspension.dae"/>
