Commit message: added wheel meshes and moved them to proper locations

File: src/uirover_description/urdf/uirover.urdf (robot description, URDF)
Before this commit: robot uirover, 16 links, 15 joints
Links:
- removed link bl_swivel
- removed link br_swivel
- removed link fl_swivel
- removed link fr_swivel
- link bl_wheel: geometry collision cylinder length=0.1 radius=0.114; visual mesh filename=file:///home/ethan/Robotics/Rover/build/uirover_description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
- link br_wheel: geometry collision cylinder length=0.1 radius=0.114; visual mesh filename=file:///home/ethan/Robotics/Rover/build/uirover_description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
- link chassis: geometry visual mesh filename=file:///home/ethan/Robotics/Rover/build/uirover_description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
- link fl_wheel: geometry collision cylinder length=0.1 radius=0.114; visual mesh filename=file:///home/ethan/Robotics/Rover/build/uirover_description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
- link fr_wheel: geometry collision cylinder length=0.1 radius=0.114; visual mesh filename=file:///home/ethan/Robotics/Rover/build/uirover_description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
- link l_suspension: geometry visual mesh filename=file:///home/ethan/Robotics/Rover/build/uirover_description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
- link ml_wheel: geometry collision cylinder length=0.1 radius=0.114; visual mesh filename=file:///home/ethan/Robotics/Rover/build/uirover_description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
- link mr_wheel: geometry collision cylinder length=0.1 radius=0.114; visual mesh filename=file:///home/ethan/Robotics/Rover/build/uirover_description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
- link r_suspension: geometry visual mesh filename=file:///home/ethan/Robotics/Rover/build/uirover_description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
Joints:
- removed joint bl_swivel_joint
- removed joint br_swivel_joint
- removed joint fl_swivel_joint
- removed joint fr_swivel_joint
- joint bl_wheel_joint: origin xyz=0 0 0 rpy=-1.5707963267948966 0 0 -> xyz=-0.434 0.1 -0.342 rpy=-1.5707963267948966 0 0; parent bl_swivel -> l_suspension
- joint br_wheel_joint: origin xyz=0 0 0 rpy=-1.5707963267948966 0 0 -> xyz=-0.434 -0.1 -0.342 rpy=-1.5707963267948966 0 0; parent br_swivel -> r_suspension
- joint fl_wheel_joint: origin xyz=0 0 0 rpy=-1.5707963267948966 0 0 -> xyz=0.436 0.1 -0.342 rpy=-1.5707963267948966 0 0; parent fl_swivel -> l_suspension
- joint fr_wheel_joint: origin xyz=0 0 0 rpy=-1.5707963267948966 0 0 -> xyz=0.436 -0.1 -0.342 rpy=-1.5707963267948966 0 0; parent fr_swivel -> r_suspension
- joint ml_wheel_joint: origin xyz=0.18 0.4 -0.35 rpy=-1.5707963267948966 0 0 -> xyz=0.016 0.1 -0.342 rpy=-1.5707963267948966 0 0; parent chassis -> l_suspension
- joint mr_wheel_joint: origin xyz=0.18 -0.4 -0.35 rpy=-1.5707963267948966 0 0 -> xyz=0.016 -0.1 -0.342 rpy=-1.5707963267948966 0 0; parent chassis -> r_suspension

File: src/uirover_description/urdf/uirover_sim.urdf (robot description, URDF)
Before this commit: robot uirover, 16 links, 15 joints
Links:
- removed link bl_swivel
- removed link br_swivel
- removed link fl_swivel
- removed link fr_swivel
- link bl_wheel: geometry collision cylinder length=0.1 radius=0.114; visual mesh filename=file:///home/ethan/Robotics/Rover/build/uirover_description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
- link br_wheel: geometry collision cylinder length=0.1 radius=0.114; visual mesh filename=file:///home/ethan/Robotics/Rover/build/uirover_description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
- link chassis: geometry visual mesh filename=file:///home/ethan/Robotics/Rover/build/uirover_description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
- link fl_wheel: geometry collision cylinder length=0.1 radius=0.114; visual mesh filename=file:///home/ethan/Robotics/Rover/build/uirover_description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
- link fr_wheel: geometry collision cylinder length=0.1 radius=0.114; visual mesh filename=file:///home/ethan/Robotics/Rover/build/uirover_description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
- link l_suspension: geometry visual mesh filename=file:///home/ethan/Robotics/Rover/build/uirover_description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
- link ml_wheel: geometry collision cylinder length=0.1 radius=0.114; visual mesh filename=file:///home/ethan/Robotics/Rover/build/uirover_description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
- link mr_wheel: geometry collision cylinder length=0.1 radius=0.114; visual mesh filename=file:///home/ethan/Robotics/Rover/build/uirover_description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
- link r_suspension: geometry visual mesh filename=file:///home/ethan/Robotics/Rover/build/uirover_description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
Joints:
- removed joint bl_swivel_joint
- removed joint br_swivel_joint
- removed joint fl_swivel_joint
- removed joint fr_swivel_joint
- joint bl_wheel_joint: origin xyz=0 0 0 rpy=-1.5707963267948966 0 0 -> xyz=-0.434 0.1 -0.342 rpy=-1.5707963267948966 0 0; parent bl_swivel -> l_suspension
- joint br_wheel_joint: origin xyz=0 0 0 rpy=-1.5707963267948966 0 0 -> xyz=-0.434 -0.1 -0.342 rpy=-1.5707963267948966 0 0; parent br_swivel -> r_suspension
- joint fl_wheel_joint: origin xyz=0 0 0 rpy=-1.5707963267948966 0 0 -> xyz=0.436 0.1 -0.342 rpy=-1.5707963267948966 0 0; parent fl_swivel -> l_suspension
- joint fr_wheel_joint: origin xyz=0 0 0 rpy=-1.5707963267948966 0 0 -> xyz=0.436 -0.1 -0.342 rpy=-1.5707963267948966 0 0; parent fr_swivel -> r_suspension
- joint ml_wheel_joint: origin xyz=0.18 0.4 -0.35 rpy=-1.5707963267948966 0 0 -> xyz=0.016 0.1 -0.342 rpy=-1.5707963267948966 0 0; parent chassis -> l_suspension
- joint mr_wheel_joint: origin xyz=0.18 -0.4 -0.35 rpy=-1.5707963267948966 0 0 -> xyz=0.016 -0.1 -0.342 rpy=-1.5707963267948966 0 0; parent chassis -> r_suspension

File: src/uirover_description/xacro/physical_description.urdf.xacro (robot description, xacro)
@@ -48,16 +48,11 @@
     <origin xyz="0.35 -0.28 0.1" rpy="0 0 0" />
   </joint>
-  <!-- SWIVEL JOINTS -->
-  <xacro:wheel_swivel name="fl_swivel" x="${chassis_length/2.5+wheel_spacing}" y="${wheel_distance_side}" z="${-suspension_height-(chassis_height/2)}" />
-  <xacro:wheel_swivel name="fr_swivel" x="${chassis_length/2.5+wheel_spacing}" y="${-wheel_distance_side}" z="${-suspension_height-(chassis_height/2)}" />
-  <xacro:wheel_swivel name="bl_swivel" x="${chassis_length/2.5-wheel_spacing}" y="${wheel_distance_side}" z="${-suspension_height-(chassis_height/2)}" />
-  <xacro:wheel_swivel name="br_swivel" x="${chassis_length/2.5-wheel_spacing}" y="${-wheel_distance_side}" z="${-suspension_height-(chassis_height/2)}" />
   <!-- WHEELS -->
-  <xacro:wheel name="fl_wheel" x="0" y="0" z ="0" parent="fl_swivel" />
-  <xacro:wheel name="fr_wheel" x="0" y="0" z ="0" parent="fr_swivel" />
-  <xacro:wheel name="ml_wheel" x="${chassis_length/2.5}" y="${wheel_distance_side}" z="${-suspension_height-(chassis_height/2)}" parent="chassis" />
-  <xacro:wheel name="mr_wheel" x="${chassis_length/2.5}" y="${-wheel_distance_side}" z="${-suspension_height-(chassis_height/2)}" parent="chassis"/>
-  <xacro:wheel name="bl_wheel" x="0" y="0" z ="0" parent="bl_swivel" />
-  <xacro:wheel name="br_wheel" x="0" y="0" z ="0" parent="br_swivel" />
+  <xacro:wheel name="fl_wheel" x="0.436"  y="0.1"  z="-0.342" parent="l_suspension" side="left"/>
+  <xacro:wheel name="fr_wheel" x="0.436"  y="-0.1" z="-0.342" parent="r_suspension" side="right"/>
+  <xacro:wheel name="ml_wheel" x="0.016"  y="0.1"  z="-0.342" parent="l_suspension" side="left"/>
+  <xacro:wheel name="mr_wheel" x="0.016"  y="-0.1" z="-0.342" parent="r_suspension" side="right"/>
+  <xacro:wheel name="bl_wheel" x="-0.434" y="0.1"  z="-0.342" parent="l_suspension" side="left"/>
+  <xacro:wheel name="br_wheel" x="-0.434" y="-0.1" z="-0.342" parent="r_suspension" side="right"/>
   <!-- Robot Footprint -->
   <!-- This is needed for nav libraries. Its the 2D top-down profile of the robot. Makes for simpler collision detection. -->

File: src/uirover_description/xacro/utility_macros.xacro (robot description, xacro)
@@ -39,13 +39,16 @@
   </xacro:macro>
   <!-- WHEEL -->
-  <xacro:macro name="wheel" params="name x y z parent">
+  <xacro:macro name="wheel" params="name x y z parent side:=^|left">
     <link name="${name}">
       <visual>
+        <xacro:if value="${side == 'left'}">
+          <origin xyz="0 0 -0.08" rpy="0 ${pi/2} 0" />
+        </xacro:if>
+        <xacro:if value="${side == 'right'}">
+          <origin xyz="0 0 0.08" rpy="0 ${-pi/2} 0" />
+        </xacro:if>
         <geometry>
-          <cylinder radius="${wheel_diameter/2}" length="${wheel_width}" />
+          <mesh filename="file://$(find uirover_description)/dae/wheel.dae"/>
         </geometry>
-        <material name="Grey">
-          <color rgba="0.7 0.7 0.7 1.0" />
-        </material>
       </visual>
       <collision>
@@ -62,30 +65,4 @@
       <origin xyz="${x} ${y} ${z}" rpy="${-pi/2} 0 0" />
       <axis xyz="0 0 1" />
-    </joint>
-  </xacro:macro>
-  <!-- WHEEL SWIVELS -->
-  <xacro:macro name="wheel_swivel" params="name x y z">
-    <link name="${name}">
-      <visual>
-        <geometry>
-          <sphere radius="0.05" />
-        </geometry>
-        <material name="Grey">
-          <color rgba="0.7 0.7 0.7 1.0" />
-        </material>
-      </visual>
-      <collision>
-        <geometry>
-          <sphere radius="0.05" />
-        </geometry>
-      </collision>
-      <xacro:box_inertia_tensor mass="0.1" len_x="0.1" len_y="0.1" len_z="0.1" />
-    </link>
-    <joint name="${name}_joint" type="revolute">
-      <parent link="base_link" />
-      <child link="${name}" />
-      <origin xyz="${x} ${y} ${z}" rpy="0 0 0" />
-      <axis xyz="0 0 1" />
-      <limit lower="${-pi/2}" upper="${pi/2}" effort="10" velocity="1" />
     </joint>
   </xacro:macro>

Commit message: rename suspension joints for consistency in URDF and Xacro files

File: src/uirover_description/urdf/uirover.urdf (robot description, URDF)
Before this commit: robot uirover, 12 links, 11 joints
Joints:
- removed joint l_suspension
- removed joint r_suspension
- added joint l_suspension_joint: type fixed, parent chassis, child l_suspension, origin xyz=0.35 0.28 0.1 rpy=0 0 0
- added joint r_suspension_joint: type fixed, parent chassis, child r_suspension, origin xyz=0.35 -0.28 0.1 rpy=0 0 0

File: src/uirover_description/urdf/uirover_sim.urdf (robot description, URDF)
Before this commit: robot uirover, 12 links, 11 joints
Joints:
- removed joint l_suspension
- removed joint r_suspension
- added joint l_suspension_joint: type fixed, parent chassis, child l_suspension, origin xyz=0.35 0.28 0.1 rpy=0 0 0
- added joint r_suspension_joint: type fixed, parent chassis, child r_suspension, origin xyz=0.35 -0.28 0.1 rpy=0 0 0

File: src/uirover_description/xacro/physical_description.urdf.xacro (robot description, xacro)
@@ -29,5 +29,5 @@
   </visual>
   </link>
-  <joint name="l_suspension" type="fixed">
+  <joint name="l_suspension_joint" type="fixed">
     <parent link="chassis" />
     <child link="l_suspension" />
@@ -43,5 +43,5 @@
   </visual>
   </link>
-  <joint name="r_suspension" type="fixed">
+  <joint name="r_suspension_joint" type="fixed">
     <parent link="chassis" />
     <child link="r_suspension" />

Commit message: Add diff drive controller configuration and update URDF/Xacro files

File: src/uirover_description/urdf/uirover.urdf (robot description, URDF)
Before this commit: robot uirover, 12 links, 11 joints
Links:
- removed link fl_wheel
- added link  , mass 0.5; collision cylinder length=0.1 radius=0.114; visual mesh filename=file:///home/ethan/Robotics/Rover/build/uirover_description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
Joints:
- removed joint fl_wheel_joint
- added joint  _joint: type continuous, parent l_suspension, child  , origin xyz=0.436 0.1 -0.342 rpy=-1.5707963267948966 0 0, axis 0 0 1

File: src/uirover_description/urdf/uirover_sim.urdf (robot description, URDF)
Before this commit: robot uirover, 12 links, 11 joints
Links:
- removed link fl_wheel
- added link  , mass 0.5; collision cylinder length=0.1 radius=0.114; visual mesh filename=file:///home/ethan/Robotics/Rover/build/uirover_description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
Joints:
- removed joint fl_wheel_joint
- added joint  _joint: type continuous, parent l_suspension, child  , origin xyz=0.436 0.1 -0.342 rpy=-1.5707963267948966 0 0, axis 0 0 1

File: src/uirover_description/xacro/gazebo.urdf.xacro (robot description, xacro)
@@ -1,9 +1,4 @@
 <?xml version="1.0"?>
 <robot name="uirover" xmlns:xacro="http://www.ros.org/wiki/xacro">
-    <!-- <gazebo>
-        <plugin filename="gz_ros2_control-system" name="gz_ros2_control::GazeboSimROS2ControlPlugin">
-            <parameters>$(find ros2_control_demo_example_9)/config/rrbot_controllers.yaml</parameters>
-        </plugin>
-    </gazebo> -->
     <!-- should probably change the color at some point. or not. orange is cool -->
     <gazebo reference="br_wheel">
@@ -25,4 +20,10 @@
         <material>Gazebo/Orange</material>
     </gazebo>
+    <gazebo reference="r_suspension">
+        <material>Gazebo/Orange</material>
+    </gazebo>
+    <gazebo reference="l_suspension">
+        <material>Gazebo/Orange</material>
+    </gazebo>
     <gazebo reference="chassis">
         <material>Gazebo/Orange</material>
@@ -31,3 +32,61 @@
         <material>Gazebo/Orange</material>
     </gazebo>
+    <ros2_control name="GazeboSimSystem" type="system">
+        <hardware>
+            <plugin>gz_ros2_control/GazeboSimSystem</plugin>
+        </hardware>
+        <joint name="fl_wheel_joint">
+            <command_interface name="velocity">
+                <param name="min">-1</param>
+                <param name="max">1</param>
+            </command_interface>
+            <state_interface name="position" />
+            <state_interface name="velocity" />
+        </joint>
+        <joint name="fr_wheel_joint">
+            <command_interface name="velocity">
+                <param name="min">-1</param>
+                <param name="max">1</param>
+            </command_interface>
+            <state_interface name="position" />
+            <state_interface name="velocity" />
+        </joint>
+        <joint name="bl_wheel_joint">
+            <command_interface name="velocity">
+                <param name="min">-1</param>
+                <param name="max">1</param>
+            </command_interface>
+            <state_interface name="position" />
+            <state_interface name="velocity" />
+        </joint>
+        <joint name="br_wheel_joint">
+            <command_interface name="velocity">
+                <param name="min">-1</param>
+                <param name="max">1</param>
+            </command_interface>
+            <state_interface name="position" />
+            <state_interface name="velocity" />
+        </joint>
+        <joint name="ml_wheel_joint">
+            <command_interface name="velocity">
+                <param name="min">-1</param>
+                <param name="max">1</param>
+            </command_interface>
+            <state_interface name="position" />
+            <state_interface name="velocity" />
+        </joint>
+        <joint name="mr_wheel_joint">
+            <command_interface name="velocity">
+                <param name="min">-1</param>
+                <param name="max">1</param>
+            </command_interface>
+            <state_interface name="position" />
+            <state_interface name="velocity" />
+        </joint>
+    </ros2_control>
+    <gazebo>
+        <plugin filename="gz_ros2_control-system" name="gz_ros2_control::GazeboSimROS2ControlPlugin">
+            <parameters>$(find uirover_description)/config/diff_drive.yaml</parameters>
+        </plugin>
+    </gazebo>
 </robot>

File: src/uirover_description/xacro/physical_description.urdf.xacro (robot description, xacro)
@@ -49,5 +49,5 @@
   </joint>
   <!-- WHEELS -->
-  <xacro:wheel name="fl_wheel" x="0.436"  y="0.1"  z="-0.342" parent="l_suspension" side="left"/>
+  <xacro:wheel name=" " x="0.436"  y="0.1"  z="-0.342" parent="l_suspension" side="left"/>
   <xacro:wheel name="fr_wheel" x="0.436"  y="-0.1" z="-0.342" parent="r_suspension" side="right"/>
   <xacro:wheel name="ml_wheel" x="0.016"  y="0.1"  z="-0.342" parent="l_suspension" side="left"/>

Commit message: added gazebo support for ros2 control

File: src/uirover_description/urdf/uirover.urdf (robot description, URDF)
Before this commit: robot uirover, 12 links, 11 joints
Links:
- removed link  
- added link fl_wheel, mass 0.5; collision cylinder length=0.1 radius=0.114; visual mesh filename=file:///home/ethan/Robotics/Rover/build/uirover_description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
Joints:
- removed joint  _joint
- added joint fl_wheel_joint: type continuous, parent l_suspension, child fl_wheel, origin xyz=0.436 0.1 -0.342 rpy=-1.5707963267948966 0 0, axis 0 0 1

File: src/uirover_description/urdf/uirover_sim.urdf (robot description, URDF)
Before this commit: robot uirover, 12 links, 11 joints
Links:
- removed link  
- added link fl_wheel, mass 0.5; collision cylinder length=0.1 radius=0.114; visual mesh filename=file:///home/ethan/Robotics/Rover/build/uirover_description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
Joints:
- removed joint  _joint
- added joint fl_wheel_joint: type continuous, parent l_suspension, child fl_wheel, origin xyz=0.436 0.1 -0.342 rpy=-1.5707963267948966 0 0, axis 0 0 1

File: src/uirover_description/urdf/uirover_sim.urdf.xacro (robot description, xacro)
@@ -4,6 +4,6 @@
     <xacro:include filename="$(find uirover_description)/xacro/physical_description.urdf.xacro"/>
     <xacro:include filename="$(find uirover_description)/xacro/sensors.urdf.xacro"/>
-    <xacro:include filename="$(find uirover_description)/xacro/ros2_control.urdf.xacro"/>
-    <xacro:uirover_ros2_control use_gazebo="true"/>
+    <!-- <xacro:include filename="$(find uirover_description)/xacro/ros2_control.urdf.xacro"/> -->
+    <!-- <xacro:uirover_ros2_control use_gazebo="true"/> -->
     <xacro:uirover_sensors use_gazebo="true"/>
 </robot>

File: src/uirover_description/xacro/gazebo.urdf.xacro (robot description, xacro)
@@ -32,5 +32,5 @@
         <material>Gazebo/Orange</material>
     </gazebo>
-    <ros2_control name="GazeboSimSystem" type="system">
+    <ros2_control name="uirover_simulator_system" type="system">
         <hardware>
             <plugin>gz_ros2_control/GazeboSimSystem</plugin>

File: src/uirover_description/xacro/physical_description.urdf.xacro (robot description, xacro)
@@ -49,5 +49,5 @@
   </joint>
   <!-- WHEELS -->
-  <xacro:wheel name=" " x="0.436"  y="0.1"  z="-0.342" parent="l_suspension" side="left"/>
+  <xacro:wheel name="fl_wheel" x="0.436"  y="0.1"  z="-0.342" parent="l_suspension" side="left"/>
   <xacro:wheel name="fr_wheel" x="0.436"  y="-0.1" z="-0.342" parent="r_suspension" side="right"/>
   <xacro:wheel name="ml_wheel" x="0.016"  y="0.1"  z="-0.342" parent="l_suspension" side="left"/>
