Commit message: cleaned up urdf/xacro files

File: src/uirover_description/urdf/uirover.urdf (robot description, URDF)
Before this commit: robot uirover, 12 links, 11 joints
Links:
- link bl_wheel: geometry collision cylinder length=0.1 radius=0.114; visual mesh filename=file:///home/ethan/Projects/Rover/build/uirover_description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
- link br_wheel: geometry collision cylinder length=0.1 radius=0.114; visual mesh filename=file:///home/ethan/Projects/Rover/build/uirover_description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
- link chassis: geometry visual mesh filename=file:///home/ethan/Projects/Rover/build/uirover_description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
- link fl_wheel: geometry collision cylinder length=0.1 radius=0.114; visual mesh filename=file:///home/ethan/Projects/Rover/build/uirover_description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
- link fr_wheel: geometry collision cylinder length=0.1 radius=0.114; visual mesh filename=file:///home/ethan/Projects/Rover/build/uirover_description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
- link l_suspension: geometry visual mesh filename=file:///home/ethan/Projects/Rover/build/uirover_description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
- link ml_wheel: geometry collision cylinder length=0.1 radius=0.114; visual mesh filename=file:///home/ethan/Projects/Rover/build/uirover_description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
- link mr_wheel: geometry collision cylinder length=0.1 radius=0.114; visual mesh filename=file:///home/ethan/Projects/Rover/build/uirover_description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
- link r_suspension: geometry visual mesh filename=file:///home/ethan/Projects/Rover/build/uirover_description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

File: src/uirover_description/urdf/uirover.urdf.xacro (robot description, xacro)
@@ -4,5 +4,3 @@
     <xacro:include filename="$(find uirover_description)/xacro/sensors.urdf.xacro"/>
     <xacro:include filename="$(find uirover_description)/xacro/ros2_control.urdf.xacro"/>
-    <xacro:uirover_ros2_control use_gazebo="false"/>
-    <xacro:uirover_sensors use_gazebo="false"/>
 </robot>

File: src/uirover_description/urdf/uirover_sim.urdf (robot description, URDF)
Before this commit: robot uirover, 12 links, 11 joints
Links:
- link bl_wheel: geometry collision cylinder length=0.1 radius=0.114; visual mesh filename=file:///home/ethan/Projects/Rover/build/uirover_description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
- link br_wheel: geometry collision cylinder length=0.1 radius=0.114; visual mesh filename=file:///home/ethan/Projects/Rover/build/uirover_description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
- link chassis: geometry visual mesh filename=file:///home/ethan/Projects/Rover/build/uirover_description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
- link fl_wheel: geometry collision cylinder length=0.1 radius=0.114; visual mesh filename=file:///home/ethan/Projects/Rover/build/uirover_description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
- link fr_wheel: geometry collision cylinder length=0.1 radius=0.114; visual mesh filename=file:///home/ethan/Projects/Rover/build/uirover_description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
- link l_suspension: geometry visual mesh filename=file:///home/ethan/Projects/Rover/build/uirover_description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
- link ml_wheel: geometry collision cylinder length=0.1 radius=0.114; visual mesh filename=file:///home/ethan/Projects/Rover/build/uirover_description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
- link mr_wheel: geometry collision cylinder length=0.1 radius=0.114; visual mesh filename=file:///home/ethan/Projects/Rover/build/uirover_description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
- link r_suspension: geometry visual mesh filename=file:///home/ethan/Projects/Rover/build/uirover_description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

File: src/uirover_description/urdf/uirover_sim.urdf.xacro (robot description, xacro)
@@ -4,6 +4,3 @@
     <xacro:include filename="$(find uirover_description)/xacro/physical_description.urdf.xacro"/>
     <xacro:include filename="$(find uirover_description)/xacro/sensors.urdf.xacro"/>
-    <!-- <xacro:include filename="$(find uirover_description)/xacro/ros2_control.urdf.xacro"/> -->
-    <!-- <xacro:uirover_ros2_control use_gazebo="true"/> -->
-    <xacro:uirover_sensors use_gazebo="true"/>
 </robot>

File: src/uirover_description/xacro/gazebo.urdf.xacro (robot description, xacro)
@@ -89,4 +89,7 @@
             <parameters>$(find uirover_description)/config/diff_drive.yaml</parameters>
         </plugin>
+        <plugin filename="gz-sim-sensors-system" name="gz::sim::systems::Sensors">
+            <render_engine>ogre2</render_engine>
+        </plugin>
     </gazebo>
 </robot>

File: src/uirover_description/xacro/ros2_control.urdf.xacro (robot description, xacro)
@@ -5,18 +5,3 @@
     <!-- https://control.ros.org/rolling/doc/getting_started/getting_started.html -->
     <!-- https://control.ros.org/rolling/doc/gz_ros2_control/doc/index.html -->
-    <xacro:macro name="uirover_ros2_control" params="use_gazebo:=^|false">
-        <ros2_control name="uirover_control" type="system" >
-            <hardware>
-                <xacro:if value="${use_gazebo}">
-                    <plugin>gz_ros2_control/GazeboSimSystem</plugin>
-                </xacro:if>
-                <!-- <xacro:unless value="${use_gazebo}">
-                    <plugin>uirover_hardware/RRBotSystemPositionOnlyHardware</plugin>
-                    <param name="example_param_hw_start_duration_sec">0</param>
-                    <param name="example_param_hw_stop_duration_sec">3.0</param>
-                    <param name="example_param_hw_slowdown">100</param>
-                </xacro:unless> -->
-            </hardware>
-        </ros2_control>
-    </xacro:macro>
 </robot>

File: src/uirover_description/xacro/sensors.urdf.xacro (robot description, xacro)
@@ -2,10 +2,9 @@
 <robot name="uirover" xmlns:xacro="http://www.ros.org/wiki/xacro">
     <xacro:include filename="$(find uirover_description)/xacro/utility_macros.xacro" />
-    <xacro:macro name="uirover_sensors" params="use_gazebo:=^|false">
         <!-- =============================== -->
         <!--            SENSORS              -->
         <!-- =============================== -->
         <!-- ARDUCAM CAMERA -->
-        <xacro:arducam name="demo_camera" use_gazebo="true" />
+        <xacro:arducam name="antenna_camera"/>
         <joint name="front_camera_joint" type="fixed">
             <origin xyz="0.0 0.2 0.8" rpy="0.0 0.5 0.0" />
@@ -13,4 +12,3 @@
             <child link="demo_camera" />
         </joint>
-    </xacro:macro>
 </robot>

File: src/uirover_description/xacro/utility_macros.xacro (robot description, xacro)
@@ -67,5 +67,5 @@
     </joint>
   </xacro:macro>
-  <xacro:macro name="arducam" params="name use_gazebo:=^|false">
+  <xacro:macro name="arducam" params="name">
     <link name="${name}">
       <visual>
@@ -91,27 +91,25 @@
       <xacro:cylinder_inertia_tensor mass="0.1" radius="0.01" length="0.01" />
     </link>
-    <xacro:if value="${use_gazebo}">
-      <gazebo reference="${name}">
-        <sensor name="boundingbox_camera" type="boundingbox_camera">
-          <topic>${name}</topic>
-          <camera>
-            <box_type>2d</box_type>
-            <!-- 110 deg FOV -->
-            <horizontal_fov>1.9198</horizontal_fov>
-            <image>
-              <width>800</width>
-              <height>600</height>
-            </image>
-            <clip>
-              <near>0.1</near>
-              <far>10</far>
-            </clip>
-          </camera>
-          <always_on>1</always_on>
-          <update_rate>30</update_rate>
-          <visualize>true</visualize>
-        </sensor>
-      </gazebo>
-    </xacro:if>
+    <gazebo reference="${name}">
+      <sensor name="boundingbox_camera" type="boundingbox_camera">
+        <topic>${name}</topic>
+        <camera>
+          <box_type>2d</box_type>
+          <!-- 110 deg FOV -->
+          <horizontal_fov>1.9198</horizontal_fov>
+          <image>
+            <width>800</width>
+            <height>600</height>
+          </image>
+          <clip>
+            <near>0.1</near>
+            <far>10</far>
+          </clip>
+        </camera>
+        <always_on>1</always_on>
+        <update_rate>30</update_rate>
+        <visualize>true</visualize>
+      </sensor>
+    </gazebo>
   </xacro:macro>
 </robot>

Commit message: Refactor camera naming and update dependencies for Gazebo integration

File: src/uirover_description/urdf/uirover.urdf (robot description, URDF)
Before this commit: robot uirover, 12 links, 11 joints
Links:
- removed link demo_camera
- added link antenna_camera, mass 0.1; collision cylinder length=0.01 radius=0.01; visual box size=0.005 0.03 0.03
- link bl_wheel: geometry collision cylinder length=0.1 radius=0.114; visual mesh filename=file:///home/ethan/Robotics/Rover/build/uirover_description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
- link br_wheel: geometry collision cylinder length=0.1 radius=0.114; visual mesh filename=file:///home/ethan/Robotics/Rover/build/uirover_description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
- link chassis: geometry visual mesh filename=file:///home/ethan/Robotics/Rover/build/uirover_description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
- link fl_wheel: geometry collision cylinder length=0.1 radius=0.114; visual mesh filename=file:///home/ethan/Robotics/Rover/build/uirover_description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
- link fr_wheel: geometry collision cylinder length=0.1 radius=0.114; visual mesh filename=file:///home/ethan/Robotics/Rover/build/uirover_description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
- link l_suspension: geometry visual mesh filename=file:///home/ethan/Robotics/Rover/build/uirover_description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
- link ml_wheel: geometry collision cylinder length=0.1 radius=0.114; visual mesh filename=file:///home/ethan/Robotics/Rover/build/uirover_description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
- link mr_wheel: geometry collision cylinder length=0.1 radius=0.114; visual mesh filename=file:///home/ethan/Robotics/Rover/build/uirover_description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
- link r_suspension: geometry visual mesh filename=file:///home/ethan/Robotics/Rover/build/uirover_description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
Joints:
- removed joint front_camera_joint
- added joint antenna_camera_joint: type fixed, parent base_link, child antenna_camera, origin xyz=0.0 0.2 0.8 rpy=0.0 0.5 0.0

File: src/uirover_description/urdf/uirover_sim.urdf (robot description, URDF)
Before this commit: robot uirover, 12 links, 11 joints
Links:
- removed link demo_camera
- added link antenna_camera, mass 0.1; collision cylinder length=0.01 radius=0.01; visual box size=0.005 0.03 0.03
- link bl_wheel: geometry collision cylinder length=0.1 radius=0.114; visual mesh filename=file:///home/ethan/Robotics/Rover/build/uirover_description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
- link br_wheel: geometry collision cylinder length=0.1 radius=0.114; visual mesh filename=file:///home/ethan/Robotics/Rover/build/uirover_description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
- link chassis: geometry visual mesh filename=file:///home/ethan/Robotics/Rover/build/uirover_description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
- link fl_wheel: geometry collision cylinder length=0.1 radius=0.114; visual mesh filename=file:///home/ethan/Robotics/Rover/build/uirover_description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
- link fr_wheel: geometry collision cylinder length=0.1 radius=0.114; visual mesh filename=file:///home/ethan/Robotics/Rover/build/uirover_description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
- link l_suspension: geometry visual mesh filename=file:///home/ethan/Robotics/Rover/build/uirover_description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
- link ml_wheel: geometry collision cylinder length=0.1 radius=0.114; visual mesh filename=file:///home/ethan/Robotics/Rover/build/uirover_description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
- link mr_wheel: geometry collision cylinder length=0.1 radius=0.114; visual mesh filename=file:///home/ethan/Robotics/Rover/build/uirover_description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
- link r_suspension: geometry visual mesh filename=file:///home/ethan/Robotics/Rover/build/uirover_description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
Joints:
- removed joint front_camera_joint
- added joint antenna_camera_joint: type fixed, parent base_link, child antenna_camera, origin xyz=0.0 0.2 0.8 rpy=0.0 0.5 0.0

File: src/uirover_description/xacro/sensors.urdf.xacro (robot description, xacro)
@@ -7,8 +7,8 @@
         <!-- ARDUCAM CAMERA -->
         <xacro:arducam name="antenna_camera"/>
-        <joint name="front_camera_joint" type="fixed">
+        <joint name="antenna_camera_joint" type="fixed">
             <origin xyz="0.0 0.2 0.8" rpy="0.0 0.5 0.0" />
             <parent link="base_link" />
-            <child link="demo_camera" />
+            <child link="antenna_camera" />
         </joint>
 </robot>

Commit message: * changed material colors * modified center of rotation * changed camera placement

File: src/uirover_description/urdf/uirover.urdf (robot description, URDF)
Before this commit: robot uirover, 12 links, 11 joints
Links:
- link bl_wheel: geometry collision cylinder length=0.1 radius=0.114; visual mesh filename=file:///home/ethan/Projects/Rover/build/uirover_description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
- link br_wheel: geometry collision cylinder length=0.1 radius=0.114; visual mesh filename=file:///home/ethan/Projects/Rover/build/uirover_description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
- link chassis: geometry visual mesh filename=file:///home/ethan/Projects/Rover/build/uirover_description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
- link fl_wheel: geometry collision cylinder length=0.1 radius=0.114; visual mesh filename=file:///home/ethan/Projects/Rover/build/uirover_description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
- link fr_wheel: geometry collision cylinder length=0.1 radius=0.114; visual mesh filename=file:///home/ethan/Projects/Rover/build/uirover_description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
- link l_suspension: geometry visual mesh filename=file:///home/ethan/Projects/Rover/build/uirover_description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
- link ml_wheel: geometry collision cylinder length=0.1 radius=0.114; visual mesh filename=file:///home/ethan/Projects/Rover/build/uirover_description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
- link mr_wheel: geometry collision cylinder length=0.1 radius=0.114; visual mesh filename=file:///home/ethan/Projects/Rover/build/uirover_description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
- link r_suspension: geometry visual mesh filename=file:///home/ethan/Projects/Rover/build/uirover_description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
Joints:
- joint antenna_camera_joint: origin xyz=0.0 0.2 0.8 rpy=0.0 0.5 0.0 -> xyz=-0.24 0.28 1.3 rpy=0.0 0.5 0.0
- joint base_footprint_joint: origin xyz=0.0 0.0 -0.44999999999999996 rpy=0 0 0 -> xyz=0.0 0.0 -0.3 rpy=0 0 0
- joint l_suspension_joint: origin xyz=0.35 0.28 0.1 rpy=0 0 0 -> xyz=0 0.28 0.1 rpy=0 0 0
- joint r_suspension_joint: origin xyz=0.35 -0.28 0.1 rpy=0 0 0 -> xyz=0 -0.28 0.1 rpy=0 0 0

File: src/uirover_description/urdf/uirover_sim.urdf (robot description, URDF)
Before this commit: robot uirover, 12 links, 11 joints
Links:
- link bl_wheel: geometry collision cylinder length=0.1 radius=0.114; visual mesh filename=file:///home/ethan/Projects/Rover/build/uirover_description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
- link br_wheel: geometry collision cylinder length=0.1 radius=0.114; visual mesh filename=file:///home/ethan/Projects/Rover/build/uirover_description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
- link chassis: geometry visual mesh filename=file:///home/ethan/Projects/Rover/build/uirover_description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
- link fl_wheel: geometry collision cylinder length=0.1 radius=0.114; visual mesh filename=file:///home/ethan/Projects/Rover/build/uirover_description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
- link fr_wheel: geometry collision cylinder length=0.1 radius=0.114; visual mesh filename=file:///home/ethan/Projects/Rover/build/uirover_description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
- link l_suspension: geometry visual mesh filename=file:///home/ethan/Projects/Rover/build/uirover_description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
- link ml_wheel: geometry collision cylinder length=0.1 radius=0.114; visual mesh filename=file:///home/ethan/Projects/Rover/build/uirover_description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
- link mr_wheel: geometry collision cylinder length=0.1 radius=0.114; visual mesh filename=file:///home/ethan/Projects/Rover/build/uirover_description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
- link r_suspension: geometry visual mesh filename=file:///home/ethan/Projects/Rover/build/uirover_description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
Joints:
- joint antenna_camera_joint: origin xyz=0.0 0.2 0.8 rpy=0.0 0.5 0.0 -> xyz=-0.24 0.28 1.3 rpy=0.0 0.5 0.0
- joint base_footprint_joint: origin xyz=0.0 0.0 -0.44999999999999996 rpy=0 0 0 -> xyz=0.0 0.0 -0.3 rpy=0 0 0
- joint l_suspension_joint: origin xyz=0.35 0.28 0.1 rpy=0 0 0 -> xyz=0 0.28 0.1 rpy=0 0 0
- joint r_suspension_joint: origin xyz=0.35 -0.28 0.1 rpy=0 0 0 -> xyz=0 -0.28 0.1 rpy=0 0 0

File: src/uirover_description/xacro/gazebo.urdf.xacro (robot description, xacro)
@@ -2,34 +2,4 @@
 <robot name="uirover" xmlns:xacro="http://www.ros.org/wiki/xacro">
     <!-- should probably change the color at some point. or not. orange is cool -->
-    <gazebo reference="br_wheel">
-        <material>Gazebo/Orange</material>
-    </gazebo>
-    <gazebo reference="bl_wheel">
-        <material>Gazebo/Orange</material>
-    </gazebo>
-    <gazebo reference="mr_wheel">
-        <material>Gazebo/Orange</material>
-    </gazebo>
-    <gazebo reference="ml_wheel">
-        <material>Gazebo/Orange</material>
-    </gazebo>
-    <gazebo reference="fr_wheel">
-        <material>Gazebo/Orange</material>
-    </gazebo>
-    <gazebo reference="fl_wheel">
-        <material>Gazebo/Orange</material>
-    </gazebo>
-    <gazebo reference="r_suspension">
-        <material>Gazebo/Orange</material>
-    </gazebo>
-    <gazebo reference="l_suspension">
-        <material>Gazebo/Orange</material>
-    </gazebo>
-    <gazebo reference="chassis">
-        <material>Gazebo/Orange</material>
-    </gazebo>
-    <gazebo reference="arm_platform">
-        <material>Gazebo/Orange</material>
-    </gazebo>
     <ros2_control name="uirover_simulator_system" type="system">
         <hardware>

File: src/uirover_description/xacro/physical_description.urdf.xacro (robot description, xacro)
@@ -9,5 +9,5 @@
   <link name="chassis">
   <visual>
-    <origin xyz="0.0 0.203 0.0" rpy="${pi/2} 0.0 0.0"/>
+    <origin xyz="-0.35 0.203 0.0" rpy="${pi/2} 0.0 0.0"/>
     <geometry>
       <mesh filename="file://$(find uirover_description)/dae/chassis.dae"/>
@@ -32,5 +32,5 @@
     <parent link="chassis" />
     <child link="l_suspension" />
-    <origin xyz="0.35 0.28 0.1" rpy="0 0 0" />
+    <origin xyz="0 0.28 0.1" rpy="0 0 0" />
   </joint>
   <!--R SUSPENSIONS-->
@@ -46,5 +46,5 @@
     <parent link="chassis" />
     <child link="r_suspension" />
-    <origin xyz="0.35 -0.28 0.1" rpy="0 0 0" />
+    <origin xyz="0 -0.28 0.1" rpy="0 0 0" />
   </joint>
   <!-- WHEELS -->
@@ -61,5 +61,5 @@
     <parent link="base_link" />
     <child link="base_footprint" />
-    <origin xyz="0.0 0.0 ${-0.3-chassis_height/2}" rpy="0 0 0" />
+    <origin xyz="0.0 0.0 -0.3" rpy="0 0 0" />
   </joint>
 </robot>

File: src/uirover_description/xacro/sensors.urdf.xacro (robot description, xacro)
@@ -8,5 +8,5 @@
         <xacro:arducam name="antenna_camera"/>
         <joint name="antenna_camera_joint" type="fixed">
-            <origin xyz="0.0 0.2 0.8" rpy="0.0 0.5 0.0" />
+            <origin xyz="-0.24 0.28 1.3" rpy="0.0 0.5 0.0" />
             <parent link="base_link" />
             <child link="antenna_camera" />
