Commit message: + gazebo terrain + added differential physics + intertia for suspension * changed gazebo physics engine * fixed covariances

File: src/uirover_description/urdf/uirover.urdf (robot description, URDF)
Before this commit: robot uirover, 12 links, 11 joints
Links:
- link l_suspension: mass None -> 2
- link r_suspension: mass None -> 2
Joints:
- joint l_suspension_joint: axis (none) -> 0 1 0; type fixed -> continuous
- joint r_suspension_joint: axis (none) -> 0 1 0; mimic (none) -> joint=l_suspension_joint multiplier=-1 offset=0; type fixed -> continuous

File: src/uirover_description/urdf/uirover_sim.urdf (robot description, URDF)
Before this commit: robot uirover, 12 links, 11 joints
Links:
- link l_suspension: mass None -> 2
- link r_suspension: mass None -> 2
Joints:
- joint l_suspension_joint: axis (none) -> 0 1 0; type fixed -> continuous
- joint r_suspension_joint: axis (none) -> 0 1 0; mimic (none) -> joint=l_suspension_joint multiplier=-1 offset=0; type fixed -> continuous

File: src/uirover_description/xacro/physical_description.urdf.xacro (robot description, xacro)
@@ -8,10 +8,10 @@
   <!-- CHASSIS -->
   <link name="chassis">
-  <visual>
-    <origin xyz="-0.35 0.203 0.0" rpy="${pi/2} 0.0 0.0"/>
-    <geometry>
-      <mesh filename="file://$(find uirover_description)/dae/chassis.dae"/>
-    </geometry>
-  </visual>
+    <visual>
+      <origin xyz="-0.35 0.203 0.0" rpy="${pi/2} 0.0 0.0" />
+      <geometry>
+        <mesh filename="file://$(find uirover_description)/dae/chassis.dae" />
+      </geometry>
+    </visual>
   </link>
   <joint name="chassis_joint" type="fixed">
@@ -20,41 +20,49 @@
     <origin xyz="0 0 0" rpy="0 0 0" />
   </joint>
-  <!--L SUSPENSIONS-->
+  <!--L
+  SUSPENSIONS-->
   <link name="l_suspension">
     <visual>
-      <origin xyz="0.085 0.02 -0.06" rpy="${pi/2} 0.0 ${pi}"/>
-    <geometry>
-      <mesh filename="file://$(find uirover_description)/dae/suspension.dae"/>
-    </geometry>
-  </visual>
+      <origin xyz="0.085 0.02 -0.06" rpy="${pi/2} 0.0 ${pi}" />
+      <geometry>
+        <mesh filename="file://$(find uirover_description)/dae/suspension.dae" />
+      </geometry>
+    </visual>
+    <xacro:box_inertia_tensor mass="2" len_x="0.65" len_y="0.05" len_z="0.15" x="0.1" y="0" z="-0.1" />
   </link>
-  <joint name="l_suspension_joint" type="fixed">
+  <joint name="l_suspension_joint" type="continuous">
     <parent link="chassis" />
     <child link="l_suspension" />
     <origin xyz="0 0.28 0.1" rpy="0 0 0" />
+    <axis xyz="0 1 0" />
   </joint>
-  <!--R SUSPENSIONS-->
+  <!--R
+  SUSPENSIONS-->
   <link name="r_suspension">
     <visual>
-      <origin xyz="0.085 0.02 -0.06" rpy="${pi/2} 0.0 ${pi}"/>
-    <geometry>
-      <mesh filename="file://$(find uirover_description)/dae/suspension.dae"/>
-    </geometry>
-  </visual>
+      <origin xyz="0.085 0.02 -0.06" rpy="${pi/2} 0.0 ${pi}" />
+      <geometry>
+        <mesh filename="file://$(find uirover_description)/dae/suspension.dae" />
+      </geometry>
+    </visual>
+    <xacro:box_inertia_tensor mass="2" len_x="0.65" len_y="0.05" len_z="0.15" x="0.1" y="0" z="-0.1" />
   </link>
-  <joint name="r_suspension_joint" type="fixed">
+  <joint name="r_suspension_joint" type="continuous">
+    <mimic joint="l_suspension_joint" multiplier="-1" offset="0" />
     <parent link="chassis" />
     <child link="r_suspension" />
     <origin xyz="0 -0.28 0.1" rpy="0 0 0" />
+    <axis xyz="0 1 0" />
   </joint>
   <!-- WHEELS -->
-  <xacro:wheel name="fl_wheel" x="0.436"  y="0.1"  z="-0.342" parent="l_suspension" side="left"/>
-  <xacro:wheel name="fr_wheel" x="0.436"  y="-0.1" z="-0.342" parent="r_suspension" side="right"/>
-  <xacro:wheel name="ml_wheel" x="0.016"  y="0.1"  z="-0.342" parent="l_suspension" side="left"/>
-  <xacro:wheel name="mr_wheel" x="0.016"  y="-0.1" z="-0.342" parent="r_suspension" side="right"/>
-  <xacro:wheel name="bl_wheel" x="-0.434" y="0.1"  z="-0.342" parent="l_suspension" side="left"/>
-  <xacro:wheel name="br_wheel" x="-0.434" y="-0.1" z="-0.342" parent="r_suspension" side="right"/>
+  <xacro:wheel name="fl_wheel" x="0.436" y="0.1" z="-0.342" parent="l_suspension" side="left" />
+  <xacro:wheel name="fr_wheel" x="0.436" y="-0.1" z="-0.342" parent="r_suspension" side="right" />
+  <xacro:wheel name="ml_wheel" x="0.016" y="0.1" z="-0.342" parent="l_suspension" side="left" />
+  <xacro:wheel name="mr_wheel" x="0.016" y="-0.1" z="-0.342" parent="r_suspension" side="right" />
+  <xacro:wheel name="bl_wheel" x="-0.434" y="0.1" z="-0.342" parent="l_suspension" side="left" />
+  <xacro:wheel name="br_wheel" x="-0.434" y="-0.1" z="-0.342" parent="r_suspension" side="right" />
   <!-- Robot Footprint -->
-  <!-- This is needed for nav libraries. Its the 2D top-down profile of the robot. Makes for simpler collision detection. -->
+  <!-- This is needed for nav libraries. Its the 2D top-down profile of the robot. Makes for simpler
+  collision detection. -->
   <link name="base_footprint" />
   <joint name="base_footprint_joint" type="fixed">

File: src/uirover_description/xacro/utility_macros.xacro (robot description, xacro)
@@ -2,5 +2,5 @@
 <robot name="uiowa_rover" xmlns:xacro="http://ros.org/wiki/xacro">
   <!-- BOX INERTIA -->
-  <xacro:macro name="box_inertia_tensor" params="mass len_x len_y len_z">
+  <xacro:macro name="box_inertia_tensor" params="mass len_x len_y len_z x y z">
     <inertial>
       <mass value="${mass}" />
@@ -8,4 +8,5 @@
         iyy="${(1/12)*mass*(len_z*len_z+len_x*len_x)}" iyz="0.0"
         izz="${(1/12)*mass*(len_x*len_x+len_y*len_y)}" />
+        <origin xyz="${x} ${y} ${z}" rpy="0 0 0" />
     </inertial>
   </xacro:macro>
@@ -104,5 +105,5 @@
           <clip>
             <near>0.1</near>
-            <far>10</far>
+            <far>100</far>
           </clip>
         </camera>

Commit message: beginning work on real hardware launch configuration

File: src/uirover_description/urdf/uirover.urdf (robot description, URDF)
Before this commit: robot uirover, 12 links, 11 joints
Links:
- link chassis: mass None -> 10; geometry collision box size=0.65 0.4 0.2; visual mesh filename=file:///home/ethan/Projects/Rover/build/uirover_description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
- link l_suspension: geometry collision box size=0.05 0.05 0.05; visual mesh filename=file:///home/ethan/Projects/Rover/build/uirover_description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
- link r_suspension: geometry collision box size=0.05 0.05 0.05; visual mesh filename=file:///home/ethan/Projects/Rover/build/uirover_description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
Joints:
- joint l_suspension_joint: type continuous -> fixed
- joint r_suspension_joint: mimic joint=l_suspension_joint multiplier=-1 offset=0 -> (none); type continuous -> fixed

File: src/uirover_description/urdf/uirover_sim.urdf (robot description, URDF)
Before this commit: robot uirover, 12 links, 11 joints
Links:
- link chassis: mass None -> 10; geometry collision box size=0.65 0.4 0.2; visual mesh filename=file:///home/ethan/Projects/Rover/build/uirover_description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
- link l_suspension: geometry collision box size=0.05 0.05 0.05; visual mesh filename=file:///home/ethan/Projects/Rover/build/uirover_description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
- link r_suspension: geometry collision box size=0.05 0.05 0.05; visual mesh filename=file:///home/ethan/Projects/Rover/build/uirover_description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
Joints:
- joint l_suspension_joint: type continuous -> fixed
- joint r_suspension_joint: mimic joint=l_suspension_joint multiplier=-1 offset=0 -> (none); type continuous -> fixed

File: src/uirover_description/xacro/physical_description.urdf.xacro (robot description, xacro)
@@ -5,5 +5,5 @@
   <xacro:include filename="$(find uirover_description)/xacro/properties.xacro" />
   <!-- BASE LINK -->
-  <link name="base_link" />
+  <link name="base_link"></link>
   <!-- CHASSIS -->
   <link name="chassis">
@@ -14,4 +14,10 @@
       </geometry>
     </visual>
+    <collision>
+      <geometry>
+        <box size="0.65 0.4 0.2" />
+      </geometry>
+    </collision>
+    <xacro:box_inertia_tensor mass="10" len_x="0.65" len_y="0.4" len_z="0.2"/>
   </link>
   <joint name="chassis_joint" type="fixed">
@@ -29,7 +35,12 @@
       </geometry>
     </visual>
+    <collision>
+      <geometry>
+        <box size="0.05 0.05 0.05" />
+      </geometry>
+    </collision>
     <xacro:box_inertia_tensor mass="2" len_x="0.65" len_y="0.05" len_z="0.15" x="0.1" y="0" z="-0.1" />
   </link>
-  <joint name="l_suspension_joint" type="continuous">
+  <joint name="l_suspension_joint" type="fixed">
     <parent link="chassis" />
     <child link="l_suspension" />
@@ -46,8 +57,13 @@
       </geometry>
     </visual>
+    <collision>
+      <geometry>
+        <box size="0.05 0.05 0.05" />
+      </geometry>
+    </collision>
     <xacro:box_inertia_tensor mass="2" len_x="0.65" len_y="0.05" len_z="0.15" x="0.1" y="0" z="-0.1" />
   </link>
-  <joint name="r_suspension_joint" type="continuous">
-    <mimic joint="l_suspension_joint" multiplier="-1" offset="0" />
+  <joint name="r_suspension_joint" type="fixed">
+    <!-- <mimic joint="l_suspension_joint" multiplier="-1" offset="0" /> -->
     <parent link="chassis" />
     <child link="r_suspension" />

File: src/uirover_description/xacro/sensors.urdf.xacro (robot description, xacro)
@@ -2,13 +2,59 @@
 <robot name="uirover" xmlns:xacro="http://www.ros.org/wiki/xacro">
     <xacro:include filename="$(find uirover_description)/xacro/utility_macros.xacro" />
-        <!-- =============================== -->
-        <!--            SENSORS              -->
-        <!-- =============================== -->
-        <!-- ARDUCAM CAMERA -->
-        <xacro:arducam name="antenna_camera"/>
-        <joint name="antenna_camera_joint" type="fixed">
-            <origin xyz="-0.24 0.28 1.3" rpy="0.0 0.5 0.0" />
-            <parent link="base_link" />
-            <child link="antenna_camera" />
-        </joint>
+    <xacro:macro name="arducam" params="name">
+        <link name="${name}">
+            <visual>
+                <origin xyz="0.0 0.0 0.0" rpy="0.0 ${pi/2} 0.0" />
+                <geometry>
+                    <cylinder radius="0.01" length="0.01" />
+                </geometry>
+                <material name="Grey">
+                    <color rgba="0.7 0.7 0.7 1.0" />
+                </material>
+            </visual>
+            <visual>
+                <origin xyz="-0.005 0.0 0.0" rpy="0.0 0.0 0.0" />
+                <geometry>
+                    <box size="0.005 0.03 0.03" />
+                </geometry>
+            </visual>
+            <collision>
+                <geometry>
+                    <cylinder radius="0.01" length="0.01" />
+                </geometry>
+            </collision>
+            <xacro:cylinder_inertia_tensor mass="0.1" radius="0.01" length="0.01" />
+        </link>
+        <gazebo reference="${name}">
+            <sensor name="camera" type="camera">
+                <topic>${name}</topic>
+                <camera>
+                    <box_type>2d</box_type>
+                    <!-- 110 deg FOV -->
+                    <horizontal_fov>1.9198</horizontal_fov>
+                    <image>
+                        <width>800</width>
+                        <height>600</height>
+                    </image>
+                    <clip>
+                        <near>0.1</near>
+                        <far>100</far>
+                    </clip>
+                </camera>
+                <always_on>1</always_on>
+                <update_rate>30</update_rate>
+                <visualize>true</visualize>
+            </sensor>
+        </gazebo>
+    </xacro:macro>
+    <!-- =============================== -->
+    <!--            SENSORS              -->
+    <!-- =============================== -->
+    <!-- ARDUCAM CAMERA -->
+    <xacro:arducam name="antenna_camera" />
+    <joint name="antenna_camera_joint" type="fixed">
+        <origin xyz="-0.24 0.28 1.3" rpy="0.0 0.5 0.0" />
+        <parent link="base_link" />
+        <child link="antenna_camera" />
+    </joint>
 </robot>

File: src/uirover_description/xacro/utility_macros.xacro (robot description, xacro)
@@ -2,5 +2,5 @@
 <robot name="uiowa_rover" xmlns:xacro="http://ros.org/wiki/xacro">
   <!-- BOX INERTIA -->
-  <xacro:macro name="box_inertia_tensor" params="mass len_x len_y len_z x y z">
+  <xacro:macro name="box_inertia_tensor" params="mass len_x len_y len_z x:=0 y:=0 z:=0">
     <inertial>
       <mass value="${mass}" />
@@ -68,49 +68,3 @@
     </joint>
   </xacro:macro>
-  <xacro:macro name="arducam" params="name">
-    <link name="${name}">
-      <visual>
-        <origin xyz="0.0 0.0 0.0" rpy="0.0 ${pi/2} 0.0" />
-        <geometry>
-          <cylinder radius="0.01" length="0.01" />
-        </geometry>
-        <material name="Grey">
-          <color rgba="0.7 0.7 0.7 1.0" />
-        </material>
-      </visual>
-      <visual>
-        <origin xyz="-0.005 0.0 0.0" rpy="0.0 0.0 0.0" />
-        <geometry>
-          <box size="0.005 0.03 0.03" />
-        </geometry>
-      </visual>
-      <collision>
-        <geometry>
-          <cylinder radius="0.01" length="0.01" />
-        </geometry>
-      </collision>
-      <xacro:cylinder_inertia_tensor mass="0.1" radius="0.01" length="0.01" />
-    </link>
-    <gazebo reference="${name}">
-      <sensor name="boundingbox_camera" type="boundingbox_camera">
-        <topic>${name}</topic>
-        <camera>
-          <box_type>2d</box_type>
-          <!-- 110 deg FOV -->
-          <horizontal_fov>1.9198</horizontal_fov>
-          <image>
-            <width>800</width>
-            <height>600</height>
-          </image>
-          <clip>
-            <near>0.1</near>
-            <far>100</far>
-          </clip>
-        </camera>
-        <always_on>1</always_on>
-        <update_rate>30</update_rate>
-        <visualize>true</visualize>
-      </sensor>
-    </gazebo>
-  </xacro:macro>
 </robot>

Commit message: refactor launch configuration

File: src/uirover_description/urdf/uirover.urdf (robot description, URDF)
Before this commit: robot uirover, 12 links, 11 joints
Links:
- link bl_wheel: geometry collision cylinder length=0.1 radius=0.114; visual mesh filename=file:///home/ethan/Robotics/Rover/build/uirover_description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
- link br_wheel: geometry collision cylinder length=0.1 radius=0.114; visual mesh filename=file:///home/ethan/Robotics/Rover/build/uirover_description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
- link chassis: geometry collision box size=0.65 0.4 0.2; visual mesh filename=file:///home/ethan/Robotics/Rover/build/uirover_description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
- link fl_wheel: geometry collision cylinder length=0.1 radius=0.114; visual mesh filename=file:///home/ethan/Robotics/Rover/build/uirover_description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
- link fr_wheel: geometry collision cylinder length=0.1 radius=0.114; visual mesh filename=file:///home/ethan/Robotics/Rover/build/uirover_description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
- link l_suspension: geometry collision box size=0.05 0.05 0.05; visual mesh filename=file:///home/ethan/Robotics/Rover/build/uirover_description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
- link ml_wheel: geometry collision cylinder length=0.1 radius=0.114; visual mesh filename=file:///home/ethan/Robotics/Rover/build/uirover_description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
- link mr_wheel: geometry collision cylinder length=0.1 radius=0.114; visual mesh filename=file:///home/ethan/Robotics/Rover/build/uirover_description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
- link r_suspension: geometry collision box size=0.05 0.05 0.05; visual mesh filename=file:///home/ethan/Robotics/Rover/build/uirover_description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

File: src/uirover_description/urdf/uirover_sim.urdf (robot description, URDF)
Before this commit: robot uirover, 12 links, 11 joints
Links:
- link bl_wheel: geometry collision cylinder length=0.1 radius=0.114; visual mesh filename=file:///home/ethan/Robotics/Rover/build/uirover_description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
- link br_wheel: geometry collision cylinder length=0.1 radius=0.114; visual mesh filename=file:///home/ethan/Robotics/Rover/build/uirover_description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
- link chassis: geometry collision box size=0.65 0.4 0.2; visual mesh filename=file:///home/ethan/Robotics/Rover/build/uirover_description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
- link fl_wheel: geometry collision cylinder length=0.1 radius=0.114; visual mesh filename=file:///home/ethan/Robotics/Rover/build/uirover_description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
- link fr_wheel: geometry collision cylinder length=0.1 radius=0.114; visual mesh filename=file:///home/ethan/Robotics/Rover/build/uirover_description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
- link l_suspension: geometry collision box size=0.05 0.05 0.05; visual mesh filename=file:///home/ethan/Robotics/Rover/build/uirover_description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
- link ml_wheel: geometry collision cylinder length=0.1 radius=0.114; visual mesh filename=file:///home/ethan/Robotics/Rover/build/uirover_description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
- link mr_wheel: geometry collision cylinder length=0.1 radius=0.114; visual mesh filename=file:///home/ethan/Robotics/Rover/build/uirover_description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
- link r_suspension: geometry collision box size=0.05 0.05 0.05; visual mesh filename=file:///home/ethan/Robotics/Rover/build/uirover_description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
