Commit message: continuing work on hardware support

File: src/uirover_description/urdf/uirover.urdf.xacro (robot description, xacro)
@@ -1,6 +1,10 @@
 <?xml version="1.0"?>
 <robot name="uirover" xmlns:xacro="http://www.ros.org/wiki/xacro">
+    <!-- Physical Description -->
     <xacro:include filename="$(find uirover_description)/xacro/physical_description.urdf.xacro"/>
+    <!-- Hardware -->
+    <xacro:include filename="$(find uirover_description)/xacro/ros2_control.urdf.xacro"/>
+    <xacro:uirover_ros2_control use_gazebo="false"/>
+    <!-- Sensors -->
     <xacro:include filename="$(find uirover_description)/xacro/sensors.urdf.xacro"/>
-    <xacro:include filename="$(find uirover_description)/xacro/ros2_control.urdf.xacro"/>
 </robot>

File: src/uirover_description/urdf/uirover_sim.urdf.xacro (robot description, xacro)
@@ -2,4 +2,6 @@
 <robot name="uirover" xmlns:xacro="http://www.ros.org/wiki/xacro">
     <xacro:include filename="$(find uirover_description)/xacro/gazebo.urdf.xacro"/>
+    <xacro:include filename="$(find uirover_description)/xacro/ros2_control.urdf.xacro"/>
+    <xacro:uirover_ros2_control use_gazebo="false"/>
     <xacro:include filename="$(find uirover_description)/xacro/physical_description.urdf.xacro"/>
     <xacro:include filename="$(find uirover_description)/xacro/sensors.urdf.xacro"/>

File: src/uirover_description/xacro/gazebo.urdf.xacro (robot description, xacro)
@@ -1,58 +1,4 @@
 <?xml version="1.0"?>
 <robot name="uirover" xmlns:xacro="http://www.ros.org/wiki/xacro">
-    <!-- should probably change the color at some point. or not. orange is cool -->
-    <ros2_control name="uirover_simulator_system" type="system">
-        <hardware>
-            <plugin>gz_ros2_control/GazeboSimSystem</plugin>
-        </hardware>
-        <joint name="fl_wheel_joint">
-            <command_interface name="velocity">
-                <param name="min">-1</param>
-                <param name="max">1</param>
-            </command_interface>
-            <state_interface name="position" />
-            <state_interface name="velocity" />
-        </joint>
-        <joint name="fr_wheel_joint">
-            <command_interface name="velocity">
-                <param name="min">-1</param>
-                <param name="max">1</param>
-            </command_interface>
-            <state_interface name="position" />
-            <state_interface name="velocity" />
-        </joint>
-        <joint name="bl_wheel_joint">
-            <command_interface name="velocity">
-                <param name="min">-1</param>
-                <param name="max">1</param>
-            </command_interface>
-            <state_interface name="position" />
-            <state_interface name="velocity" />
-        </joint>
-        <joint name="br_wheel_joint">
-            <command_interface name="velocity">
-                <param name="min">-1</param>
-                <param name="max">1</param>
-            </command_interface>
-            <state_interface name="position" />
-            <state_interface name="velocity" />
-        </joint>
-        <joint name="ml_wheel_joint">
-            <command_interface name="velocity">
-                <param name="min">-1</param>
-                <param name="max">1</param>
-            </command_interface>
-            <state_interface name="position" />
-            <state_interface name="velocity" />
-        </joint>
-        <joint name="mr_wheel_joint">
-            <command_interface name="velocity">
-                <param name="min">-1</param>
-                <param name="max">1</param>
-            </command_interface>
-            <state_interface name="position" />
-            <state_interface name="velocity" />
-        </joint>
-    </ros2_control>
     <gazebo>
         <plugin filename="gz_ros2_control-system" name="gz_ros2_control::GazeboSimROS2ControlPlugin">

File: src/uirover_description/xacro/ros2_control.urdf.xacro (robot description, xacro)
@@ -5,3 +5,53 @@
     <!-- https://control.ros.org/rolling/doc/getting_started/getting_started.html -->
     <!-- https://control.ros.org/rolling/doc/gz_ros2_control/doc/index.html -->
+    <xacro:macro name="uirover_ros2_control" params="use_gazebo:=^|false">
+        <ros2_control name="uirover_hardware_system" type="system">
+            <!-- Hardware Plugin -->
+            <hardware>
+                <xacro:if value="${use_gazebo}">
+                    <plugin>gz_ros2_control/GazeboSimSystem</plugin>
+                </xacro:if>
+                <xacro:unless value="${use_gazebo}">
+                    <plugin>uirover_hardware/UiroverHardwareInterface</plugin>
+                </xacro:unless>
+            </hardware>
+            <!-- Joints -->
+            <joint name="fl_wheel_joint">
+                <command_interface name="velocity">
+                    <param name="min">-1</param>
+                    <param name="max">1</param>
+                </command_interface>
+            </joint>
+            <joint name="fr_wheel_joint">
+                <command_interface name="velocity">
+                    <param name="min">-1</param>
+                    <param name="max">1</param>
+                </command_interface>
+            </joint>
+            <joint name="bl_wheel_joint">
+                <command_interface name="velocity">
+                    <param name="min">-1</param>
+                    <param name="max">1</param>
+                </command_interface>
+            </joint>
+            <joint name="br_wheel_joint">
+                <command_interface name="velocity">
+                    <param name="min">-1</param>
+                    <param name="max">1</param>
+                </command_interface>
+            </joint>
+            <joint name="ml_wheel_joint">
+                <command_interface name="velocity">
+                    <param name="min">-1</param>
+                    <param name="max">1</param>
+                </command_interface>
+            </joint>
+            <joint name="mr_wheel_joint">
+                <command_interface name="velocity">
+                    <param name="min">-1</param>
+                    <param name="max">1</param>
+                </command_interface>
+            </joint>
+        </ros2_control>
+    </xacro:macro>
 </robot>

Commit message: added arm description and moveit2 configuration

File: src/uirover_description/urdf/uirover.urdf.xacro (robot description, xacro)
@@ -2,5 +2,5 @@
 <robot name="uirover" xmlns:xacro="http://www.ros.org/wiki/xacro">
     <!-- Physical Description -->
-    <xacro:include filename="$(find uirover_description)/xacro/physical_description.urdf.xacro"/>
+    <xacro:include filename="$(find uirover_description)/xacro/chassis.urdf.xacro"/>
     <!-- Hardware -->
     <xacro:include filename="$(find uirover_description)/xacro/ros2_control.urdf.xacro"/>
@@ -8,3 +8,5 @@
     <!-- Sensors -->
     <xacro:include filename="$(find uirover_description)/xacro/sensors.urdf.xacro"/>
+    <!-- Arm -->
+    <xacro:include filename="$(find uirover_description)/xacro/arm.urdf.xacro"/>
 </robot>

File: src/uirover_description/urdf/uirover_sim.urdf.xacro (robot description, xacro)
@@ -4,5 +4,5 @@
     <xacro:include filename="$(find uirover_description)/xacro/ros2_control.urdf.xacro"/>
     <xacro:uirover_ros2_control use_gazebo="false"/>
-    <xacro:include filename="$(find uirover_description)/xacro/physical_description.urdf.xacro"/>
+    <xacro:include filename="$(find uirover_description)/xacro/chassis.urdf.xacro"/>
     <xacro:include filename="$(find uirover_description)/xacro/sensors.urdf.xacro"/>
 </robot>

File: src/uirover_description/xacro/chassis.urdf.xacro (robot description, xacro)
@@ -16,8 +16,15 @@
     <collision>
       <geometry>
-        <box size="0.65 0.4 0.2" />
+        <box size="0.45 0.45 0.3" />
       </geometry>
+      <origin xyz="-0.12 0 0.15" />
     </collision>
-    <xacro:box_inertia_tensor mass="10" len_x="0.65" len_y="0.4" len_z="0.2"/>
+    <collision>
+      <geometry>
+        <box size="0.25 0.45 0.03" />
+      </geometry>
+      <origin xyz="0.23 0 0.01"/>
+    </collision>
+    <xacro:box_inertia_tensor mass="10" len_x="0.65" len_y="0.4" len_z="0.2" />
   </link>
   <joint name="chassis_joint" type="fixed">

File: src/uirover_description/xacro/properties.xacro (robot description, xacro)
@@ -1,4 +1,4 @@
 <?xml version="1.0" encoding="UTF-8"?>
-<robot name="uiowa_rover" xmlns:xacro="http://ros.org/wiki/xacro">
+<robot name="uirover" xmlns:xacro="http://ros.org/wiki/xacro">
     <xacro:property name="wheel_diameter" value="0.23" />
     <xacro:property name="chassis_width" value="0.45" />

File: src/uirover_description/xacro/utility_macros.xacro (robot description, xacro)
@@ -1,4 +1,4 @@
 <?xml version="1.0" encoding="UTF-8"?>
-<robot name="uiowa_rover" xmlns:xacro="http://ros.org/wiki/xacro">
+<robot name="uirover" xmlns:xacro="http://ros.org/wiki/xacro">
   <!-- BOX INERTIA -->
   <xacro:macro name="box_inertia_tensor" params="mass len_x len_y len_z x:=0 y:=0 z:=0">

Commit message: Add CAN bus interface and update hardware configurations
- Introduced uirover_canbus_interface for CAN communication.
- Updated CMakeLists.txt to include the new interface.
- Modified XML configurations for ros2_control to use CANInterface.
- Updated MoveIt configs
- Cleaned up .gitignore and removed obsolete test files.

File: src/uirover_description/urdf/uirover.urdf.xacro (robot description, xacro)
@@ -4,6 +4,6 @@
     <xacro:include filename="$(find uirover_description)/xacro/chassis.urdf.xacro"/>
     <!-- Hardware -->
-    <xacro:include filename="$(find uirover_description)/xacro/ros2_control.urdf.xacro"/>
-    <xacro:uirover_ros2_control use_gazebo="false"/>
+    <!-- <xacro:include filename="$(find uirover_description)/xacro/ros2_control.urdf.xacro"/> -->
+    <!-- <xacro:uirover_ros2_control use_gazebo="false"/> -->
     <!-- Sensors -->
     <xacro:include filename="$(find uirover_description)/xacro/sensors.urdf.xacro"/>

File: src/uirover_description/xacro/ros2_control.urdf.xacro (robot description, xacro)
@@ -13,5 +13,6 @@
                 </xacro:if>
                 <xacro:unless value="${use_gazebo}">
-                    <plugin>uirover_hardware/UiroverHardwareInterface</plugin>
+                    <!-- <plugin>uirover_hardware/UiroverHardwareInterface</plugin> -->
+                    <plugin>mock_components/GenericSystem</plugin>
                 </xacro:unless>
             </hardware>

File: src/uirover_moveit/config/uirover.ros2_control.xacro (robot description, xacro)
@@ -2,51 +2,45 @@
 <robot xmlns:xacro="http://www.ros.org/wiki/xacro">
     <xacro:macro name="uirover_ros2_control" params="name initial_positions_file">
-        <xacro:property name="initial_positions" value="${xacro.load_yaml(initial_positions_file)['initial_positions']}"/>
         <ros2_control name="${name}" type="system">
             <hardware>
                 <!-- By default, set up controllers for simulation. This won't work on real hardware -->
-                <plugin>mock_components/GenericSystem</plugin>
+                 <!-- TODO set correct serial numbers -->
+                <plugin>uirover_hardware/CANInterface</plugin>
             </hardware>
             <joint name="arm_j0">
                 <command_interface name="position"/>
-                <state_interface name="position">
-                  <param name="initial_value">${initial_positions['arm_j0']}</param>
-                </state_interface>
+                <state_interface name="position"/>
                 <state_interface name="velocity"/>
+                <param name="odrive_serial_number">100</param>
             </joint>
             <joint name="arm_j1">
                 <command_interface name="position"/>
-                <state_interface name="position">
-                  <param name="initial_value">${initial_positions['arm_j1']}</param>
-                </state_interface>
+                <state_interface name="position"/>
                 <state_interface name="velocity"/>
+                <param name="odrive_serial_number">101</param>
             </joint>
             <joint name="arm_j2">
                 <command_interface name="position"/>
-                <state_interface name="position">
-                  <param name="initial_value">${initial_positions['arm_j2']}</param>
-                </state_interface>
+                <state_interface name="position"/>
                 <state_interface name="velocity"/>
+                <param name="odrive_serial_number">102</param>
             </joint>
             <joint name="arm_j3">
                 <command_interface name="position"/>
-                <state_interface name="position">
-                  <param name="initial_value">${initial_positions['arm_j3']}</param>
-                </state_interface>
+                <state_interface name="position"/>
                 <state_interface name="velocity"/>
+                <param name="odrive_serial_number">103</param>
             </joint>
             <joint name="arm_j4">
                 <command_interface name="position"/>
-                <state_interface name="position">
-                  <param name="initial_value">${initial_positions['arm_j4']}</param>
-                </state_interface>
+                <state_interface name="position"/>
                 <state_interface name="velocity"/>
+                <param name="odrive_serial_number">104</param>
             </joint>
             <joint name="arm_j5">
                 <command_interface name="position"/>
-                <state_interface name="position">
-                  <param name="initial_value">${initial_positions['arm_j5']}</param>
-                </state_interface>
+                <state_interface name="position"/>
                 <state_interface name="velocity"/>
+                <param name="odrive_serial_number">105</param>
             </joint>
         </ros2_control>

File: src/uirover_moveit/config/uirover.urdf.xacro (robot description, xacro)
@@ -6,4 +6,4 @@
     <!-- Import control_xacro -->
     <xacro:include filename="uirover.ros2_control.xacro" />
-    <xacro:uirover_ros2_control name="FakeSystem" initial_positions_file="$(arg initial_positions_file)"/>
+    <xacro:uirover_ros2_control name="CANBusArm" initial_positions_file="$(arg initial_positions_file)"/>
 </robot>

Commit message: Refactor uirover_hardware interface and CAN bus communication
- Removed visibility control macros from UiroverHardwareInterface.
- Simplified the send_cmd function in CANInterface by removing the length parameter and hardcoding the data length to 8.
- Updated the CAN interface to use "vcan0" instead of "can0".
- Adjusted the command sending logic for Odrive to match the new send_cmd signature.

Update MoveIt configuration and launch files

- Added end_effector controller to moveit_controllers.yaml.
- Updated moveit.rviz configuration to streamline visualization settings.
- Created a new launch file for MoveIt integration with uirover, including necessary nodes and parameters.
- Adjusted URDF and XACRO files to support mock and target hardware configurations.

Enhance uirover_moveit configuration files

- Added initial position parameters for arm joints in uirover.ros2_control.xacro.
- Removed unnecessary group states from uirover.srdf.
- Updated the RViz configuration to improve visualization and interaction settings.
- Created a default RViz configuration file for uirover_basestation.

General improvements and cleanup

- Cleaned up code and comments across various files for better readability and maintainability.
- Ensured all configuration files are consistent with the latest changes in the hardware interface and MoveIt setup.

File: src/uirover_description/urdf/uirover.urdf.xacro (robot description, xacro)
@@ -1,12 +1,12 @@
 <?xml version="1.0"?>
-<robot name="uirover" xmlns:xacro="http://www.ros.org/wiki/xacro">
-    <!-- Physical Description -->
-    <xacro:include filename="$(find uirover_description)/xacro/chassis.urdf.xacro"/>
-    <!-- Hardware -->
-    <!-- <xacro:include filename="$(find uirover_description)/xacro/ros2_control.urdf.xacro"/> -->
-    <!-- <xacro:uirover_ros2_control use_gazebo="false"/> -->
-    <!-- Sensors -->
-    <xacro:include filename="$(find uirover_description)/xacro/sensors.urdf.xacro"/>
-    <!-- Arm -->
-    <xacro:include filename="$(find uirover_description)/xacro/arm.urdf.xacro"/>
+<robot name="uirover"
+    xmlns:xacro="http://www.ros.org/wiki/xacro">
+        <!-- Chassis -->
+        <xacro:include filename="$(find uirover_description)/xacro/chassis.urdf.xacro"/>
+        <!-- Arm -->
+        <xacro:include filename="$(find uirover_description)/xacro/arm.urdf.xacro"/>
+        <!-- Hardware -->
+        <xacro:include filename="$(find uirover_hardware)/xacro/ros2_control.urdf.xacro"/>
+        <!-- Sensors -->
+        <xacro:include filename="$(find uirover_description)/xacro/sensors.urdf.xacro"/>
 </robot>

File: src/uirover_description/urdf/uirover_sim.urdf.xacro (robot description, xacro)
@@ -2,6 +2,6 @@
 <robot name="uirover" xmlns:xacro="http://www.ros.org/wiki/xacro">
     <xacro:include filename="$(find uirover_description)/xacro/gazebo.urdf.xacro"/>
-    <xacro:include filename="$(find uirover_description)/xacro/ros2_control.urdf.xacro"/>
-    <xacro:uirover_ros2_control use_gazebo="true"/>
+    <xacro:include filename="$(find uirover_hardware)/xacro/ros2_control.urdf.xacro"/>
+    <xacro:uirover_ros2_control hw_type="target"/>
     <xacro:include filename="$(find uirover_description)/xacro/chassis.urdf.xacro"/>
     <xacro:include filename="$(find uirover_description)/xacro/sensors.urdf.xacro"/>

File: src/uirover_description/xacro/utility_macros.xacro (robot description, xacro)
@@ -61,9 +61,9 @@
         length="${wheel_width}" />
     </link>
-    <joint name="${name}_joint" type="fixed">
+    <joint name="${name}_joint" type="continuous">
       <parent link="${parent}" />
       <child link="${name}" />
       <origin xyz="${x} ${y} ${z}" rpy="${-pi/2} 0 0" />
-      <!-- <axis xyz="0 0 1" /> -->
+      <axis xyz="0 0 1" />
     </joint>
   </xacro:macro>

File: src/uirover_moveit/config/uirover.ros2_control.xacro (robot description, xacro)
@@ -2,45 +2,51 @@
 <robot xmlns:xacro="http://www.ros.org/wiki/xacro">
     <xacro:macro name="uirover_ros2_control" params="name initial_positions_file">
+        <xacro:property name="initial_positions" value="${xacro.load_yaml(initial_positions_file)['initial_positions']}"/>
         <ros2_control name="${name}" type="system">
             <hardware>
                 <!-- By default, set up controllers for simulation. This won't work on real hardware -->
-                 <!-- TODO set correct serial numbers -->
-                <plugin>uirover_hardware/CANInterface</plugin>
+                <plugin>mock_components/GenericSystem</plugin>
             </hardware>
             <joint name="arm_j0">
                 <command_interface name="position"/>
-                <state_interface name="position"/>
+                <state_interface name="position">
+                  <param name="initial_value">${initial_positions['arm_j0']}</param>
+                </state_interface>
                 <state_interface name="velocity"/>
-                <param name="odrive_serial_number">C0FFEE00</param>
             </joint>
             <joint name="arm_j1">
                 <command_interface name="position"/>
-                <state_interface name="position"/>
+                <state_interface name="position">
+                  <param name="initial_value">${initial_positions['arm_j1']}</param>
+                </state_interface>
                 <state_interface name="velocity"/>
-                <param name="odrive_serial_number">C0FFEE01</param>
             </joint>
             <joint name="arm_j2">
                 <command_interface name="position"/>
-                <state_interface name="position"/>
+                <state_interface name="position">
+                  <param name="initial_value">${initial_positions['arm_j2']}</param>
+                </state_interface>
                 <state_interface name="velocity"/>
-                <param name="odrive_serial_number">C0FFEE02</param>
             </joint>
             <joint name="arm_j3">
                 <command_interface name="position"/>
-                <state_interface name="position"/>
+                <state_interface name="position">
+                  <param name="initial_value">${initial_positions['arm_j3']}</param>
+                </state_interface>
                 <state_interface name="velocity"/>
-                <param name="odrive_serial_number">C0FFEE03</param>
             </joint>
             <joint name="arm_j4">
                 <command_interface name="position"/>
-                <state_interface name="position"/>
+                <state_interface name="position">
+                  <param name="initial_value">${initial_positions['arm_j4']}</param>
+                </state_interface>
                 <state_interface name="velocity"/>
-                <param name="odrive_serial_number">C0FFEE04</param>
             </joint>
             <joint name="arm_j5">
                 <command_interface name="position"/>
-                <state_interface name="position"/>
+                <state_interface name="position">
+                  <param name="initial_value">${initial_positions['arm_j5']}</param>
+                </state_interface>
                 <state_interface name="velocity"/>
-                <param name="odrive_serial_number">C0FFEE05</param>
             </joint>
         </ros2_control>

File: src/uirover_moveit/config/uirover.urdf.xacro (robot description, xacro)
@@ -6,4 +6,4 @@
     <!-- Import control_xacro -->
     <xacro:include filename="uirover.ros2_control.xacro" />
-    <xacro:uirover_ros2_control name="CANBusArm" initial_positions_file="$(arg initial_positions_file)"/>
+    <xacro:uirover_ros2_control name="FakeSystem" initial_positions_file="$(arg initial_positions_file)"/>
 </robot>
