Commit message: integrated gazebo into main launch file as a configuration. other minor changes

File: src/uirover_description/urdf/uirover.urdf.xacro (robot description, xacro)
@@ -2,11 +2,11 @@
 <robot name="uirover"
     xmlns:xacro="http://www.ros.org/wiki/xacro">
-        <!-- Chassis -->
-        <xacro:include filename="$(find uirover_description)/xacro/chassis.urdf.xacro"/>
-        <!-- Arm -->
-        <xacro:include filename="$(find uirover_description)/xacro/arm.urdf.xacro"/>
-        <!-- Hardware -->
-        <xacro:include filename="$(find uirover_hardware)/xacro/ros2_control.urdf.xacro"/>
-        <!-- Sensors -->
-        <xacro:include filename="$(find uirover_description)/xacro/sensors.urdf.xacro"/>
+    <!-- Chassis -->
+    <xacro:include filename="$(find uirover_description)/xacro/chassis.urdf.xacro"/>
+    <!-- Arm -->
+    <xacro:include filename="$(find uirover_description)/xacro/arm.urdf.xacro"/>
+    <!-- Hardware -->
+    <xacro:include filename="$(find uirover_hardware)/xacro/ros2_control.urdf.xacro"/>
+    <!-- Sensors -->
+    <xacro:include filename="$(find uirover_description)/xacro/sensors.urdf.xacro"/>
 </robot>

File: src/uirover_description/xacro/arm.urdf.xacro (robot description, xacro)
@@ -23,4 +23,10 @@
             <origin xyz="0 0 0.11" rpy="${pi/2} 0 0" />
         </collision>
+        <!-- approximate inertial (mass ~1.0 kg) computed from main cylinder collision -->
+        <inertial>
+            <origin xyz="0 0 0.11" rpy="${pi/2} 0 0" />
+            <mass value="1.0"/>
+            <inertia ixx="0.002533" ixy="0.0" ixz="0.0" iyy="0.002533" iyz="0.0" izz="0.001800"/>
+        </inertial>
     </link>
     <joint name="arm_j0" type="revolute">
@@ -50,4 +56,10 @@
             <origin xyz="0 -0.02 0.53" rpy="${pi/2} 0 0" />
         </collision>
+        <!-- approximate inertial (mass ~2.0 kg) using main long cylinder -->
+        <inertial>
+            <origin xyz="0 0 0.27" rpy="0 0 0" />
+            <mass value="2.0"/>
+            <inertia ixx="0.024517" ixy="0.0" ixz="0.0" iyy="0.024517" iyz="0.0" izz="0.000900"/>
+        </inertial>
     </link>
     <joint name="arm_j1" type="revolute">
@@ -77,4 +89,10 @@
             <origin xyz="0 0.08 0.1" rpy="0 0 0" />
         </collision>
+        <!-- approximate inertial (mass ~1.5 kg) using larger-radius cylinder -->
+        <inertial>
+            <origin xyz="0 0.08 -0.005" rpy="${pi/2} 0 0" />
+            <mass value="1.5"/>
+            <inertia ixx="0.001934" ixy="0.0" ixz="0.0" iyy="0.001934" iyz="0.0" izz="0.002269"/>
+        </inertial>
     </link>
     <joint name="arm_j2" type="revolute">
@@ -110,4 +128,10 @@
             <origin xyz="0 0.03 0.18" rpy="${pi/2} 0 0" />
         </collision>
+        <!-- approximate inertial (mass ~1.5 kg) using larger cylinder/combined geometry -->
+        <inertial>
+            <origin xyz="0 0 0" rpy="0 ${pi/2} 0" />
+            <mass value="1.5"/>
+            <inertia ixx="0.002384" ixy="0.0" ixz="0.0" iyy="0.002384" iyz="0.0" izz="0.002269"/>
+        </inertial>
     </link>
     <joint name="arm_j3" type="revolute">
@@ -131,4 +155,10 @@
             <origin xyz="0 -0.075 0" rpy="0 0 0" />
         </collision>
+        <!-- approximate inertial (mass ~0.7 kg) using main cylinder -->
+        <inertial>
+            <origin xyz="0 -0.075 0" rpy="0 0 0" />
+            <mass value="0.7"/>
+            <inertia ixx="0.001470" ixy="0.0" ixz="0.0" iyy="0.001470" iyz="0.0" izz="0.001260"/>
+        </inertial>
     </link>
     <joint name="arm_j4" type="revolute">
@@ -152,4 +182,10 @@
             <origin xyz="0 0 0.03" rpy="0 0 0" />
         </collision>
+        <!-- approximate inertial (mass ~0.2 kg) small end link -->
+        <inertial>
+            <origin xyz="0 0 0.03" rpy="0 0 0" />
+            <mass value="0.2"/>
+            <inertia ixx="0.000222" ixy="0.0" ixz="0.0" iyy="0.000222" iyz="0.0" izz="0.000360"/>
+        </inertial>
     </link>
     <joint name="arm_j5" type="continuous">
@@ -174,4 +210,10 @@
             <origin xyz="0 0 -0.05" rpy="0 0 0" />
         </collision>
+        <!-- approximate inertial (mass ~0.1 kg) for small end effector box -->
+        <inertial>
+            <origin xyz="0 0 -0.05" rpy="0 0 0" />
+            <mass value="0.1"/>
+            <inertia ixx="8.6667e-05" ixy="0.0" ixz="0.0" iyy="8.6667e-05" iyz="0.0" izz="6.6667e-06"/>
+        </inertial>
     </link>
     <joint name="end_effector_joint" type="fixed">

File: src/uirover_hardware/xacro/ros2_control.urdf.xacro (robot description, xacro)
@@ -1,7 +1,19 @@
 <?xml version="1.0"?>
-<robot name="uirover" xmlns:xacro="http://www.ros.org/wiki/xacro">
+<robot name="uirover"
+    xmlns:xacro="http://www.ros.org/wiki/xacro">
     <xacro:arg name="hw_type" default="target"/>
     <xacro:property name='hw_type' value="$(arg hw_type)"/>
-    <ros2_control name="wheels" type="system">
+    <gazebo>
+        <plugin filename="gz_ros2_control-system" name="gz_ros2_control::GazeboSimROS2ControlPlugin">
+            <ros>
+                <namespace>/uirover/control</namespace>
+            </ros>
+            <parameters>$(find uirover_controllers)/config/controllers.yaml</parameters>
+        </plugin>
+        <plugin filename="gz-sim-sensors-system" name="gz::sim::systems::Sensors">
+            <render_engine>ogre2</render_engine>
+        </plugin>
+    </gazebo>
+    <ros2_control name="wheels_hardware" type="system">
         <hardware>
             <xacro:if value="${hw_type=='gazebo'}">
@@ -21,4 +33,5 @@
             </command_interface>
             <state_interface name="velocity" />
+            <state_interface name="position" />
         </joint>
         <joint name="fr_wheel_joint">
@@ -28,4 +41,5 @@
             </command_interface>
             <state_interface name="velocity" />
+            <state_interface name="position" />
         </joint>
         <joint name="bl_wheel_joint">
@@ -35,4 +49,5 @@
             </command_interface>
             <state_interface name="velocity" />
+            <state_interface name="position" />
         </joint>
         <joint name="br_wheel_joint">
@@ -42,4 +57,5 @@
             </command_interface>
             <state_interface name="velocity" />
+            <state_interface name="position" />
         </joint>
         <joint name="ml_wheel_joint">
@@ -49,4 +65,5 @@
             </command_interface>
             <state_interface name="velocity" />
+            <state_interface name="position" />
         </joint>
         <joint name="mr_wheel_joint">
@@ -56,7 +73,8 @@
             </command_interface>
             <state_interface name="velocity" />
+            <state_interface name="position" />
         </joint>
     </ros2_control>
-    <ros2_control name="arm" type="system" params="hw_type:='target'">
+    <ros2_control name="arm_hardware" type="system" params="hw_type:='target'">
         <hardware>
             <!-- Hardware plugin for Gazebo Sim -->
@@ -75,5 +93,5 @@
         <joint name="arm_j0">
             <command_interface name="position" />
-            <state_interface name="position" >
+            <state_interface name="position">
                 <param name="initial_value">0.0</param>
             </state_interface>
@@ -83,6 +101,6 @@
         <joint name="arm_j1">
             <command_interface name="position" />
-            <state_interface name="position" >
-                <param name="initial_value">15.0</param>
+            <state_interface name="position">
+                <param name="initial_value">0.262</param>
             </state_interface>
             <state_interface name="velocity" />
@@ -91,6 +109,6 @@
         <joint name="arm_j2">
             <command_interface name="position" />
-            <state_interface name="position" >
-                <param name="initial_value">100.0</param>
+            <state_interface name="position">
+                <param name="initial_value">1.745</param>
             </state_interface>
             <state_interface name="velocity" />
@@ -99,5 +117,5 @@
         <joint name="arm_j3">
             <command_interface name="position" />
-            <state_interface name="position" >
+            <state_interface name="position">
                 <param name="initial_value">0.0</param>
             </state_interface>
@@ -107,6 +125,6 @@
         <joint name="arm_j4">
             <command_interface name="position" />
-            <state_interface name="position" >
-                <param name="initial_value">-25.0</param>
+            <state_interface name="position">
+                <param name="initial_value">-0.436</param>
             </state_interface>
             <state_interface name="velocity" />
@@ -115,5 +133,5 @@
         <joint name="arm_j5">
             <command_interface name="position" />
-            <state_interface name="position" >
+            <state_interface name="position">
                 <param name="initial_value">0.0</param>
             </state_interface>

Commit message: Refactor launch files and URDF configurations for improved simulation support; added GPS sensor and updated inertia properties.

File: src/uirover_description/urdf/uirover.urdf.xacro (robot description, xacro)
@@ -2,4 +2,5 @@
 <robot name="uirover"
     xmlns:xacro="http://www.ros.org/wiki/xacro">
+    <!-- https://wiki.ros.org/urdf/XML -->
     <!-- Chassis -->
     <xacro:include filename="$(find uirover_description)/xacro/chassis.urdf.xacro"/>
@@ -10,3 +11,4 @@
     <!-- Sensors -->
     <xacro:include filename="$(find uirover_description)/xacro/sensors.urdf.xacro"/>
+    <xacro:include filename="$(find uirover_description)/xacro/gazebo.urdf.xacro"/>
 </robot>

File: src/uirover_description/xacro/chassis.urdf.xacro (robot description, xacro)
@@ -26,5 +26,5 @@
       <origin xyz="0.23 0 0.01"/>
     </collision>
-    <xacro:box_inertia_tensor mass="10" len_x="0.65" len_y="0.4" len_z="0.2" />
+    <xacro:box_inertia_tensor mass="30" len_x="0.65" len_y="0.4" len_z="0.2" />
   </link>
   <joint name="chassis_joint" type="fixed">

File: src/uirover_description/xacro/gazebo.urdf.xacro (robot description, xacro)
@@ -1,11 +1,17 @@
 <?xml version="1.0"?>
-<robot name="uirover" xmlns:xacro="http://www.ros.org/wiki/xacro">
+<robot name="uirover"
+    xmlns:xacro="http://www.ros.org/wiki/xacro">
     <gazebo>
         <plugin filename="gz_ros2_control-system" name="gz_ros2_control::GazeboSimROS2ControlPlugin">
-            <parameters>$(find uirover_description)/config/diff_drive.yaml</parameters>
+            <ros>
+                <namespace>/uirover/control</namespace>
+            </ros>
+            <parameters>$(find uirover_controllers)/config/controllers.yaml</parameters>
         </plugin>
         <plugin filename="gz-sim-sensors-system" name="gz::sim::systems::Sensors">
             <render_engine>ogre2</render_engine>
         </plugin>
+        <plugin filename="gz-sim-sensors-navsat" name="gz::sim::systems::NavSat">
+        </plugin>
     </gazebo>
 </robot>

File: src/uirover_description/xacro/sensors.urdf.xacro (robot description, xacro)
@@ -1,4 +1,5 @@
 <?xml version="1.0"?>
-<robot name="uirover" xmlns:xacro="http://www.ros.org/wiki/xacro">
+<robot name="uirover"
+    xmlns:xacro="http://www.ros.org/wiki/xacro">
     <xacro:include filename="$(find uirover_description)/xacro/utility_macros.xacro" />
     <xacro:macro name="arducam" params="name">
@@ -58,3 +59,44 @@
         <child link="antenna_camera" />
     </joint>
+    <link name="ZED_F9P_GPS">
+        <gazebo reference="ZED_F9P_GPS">
+            <sensor name="ZED_F9P_GPS" type="navsat">
+                <navsat>
+                    <position_sensing>
+                        <horizontal>
+                            <noise type="gaussian">
+                                <mean>0</mean>
+                                <stddev>1.75e-6</stddev>
+                            </noise>
+                        </horizontal>
+                        <vertical>
+                            <noise type="gaussian">
+                                <mean>0.0</mean>
+                                <stddev>1.35e-6</stddev>
+                            </noise>
+                        </vertical>
+                    </position_sensing>
+                    <vertical_sensing>
+                        <horizontal>
+                            <noise type="gaussian">
+                                <mean>0.0</mean>
+                                <stddev>0.0001</stddev>
+                            </noise>
+                        </horizontal>
+                        <vertical>
+                            <noise type="gaussian">
+                                <mean>0.0</mean>
+                                <stddev>0.0001</stddev>
+                            </noise>
+                        </vertical>
+                    </vertical_sensing>
+                </navsat>
+            </sensor>
+        </gazebo>
+    </link>
+    <joint name="ZED_F9P_GPS_joint" type="fixed">
+        <origin xyz="0 0 0"/>
+        <parent link="base_link"/>
+        <child link="ZED_F9P_GPS"/>
+    </joint>
 </robot>

File: src/uirover_description/xacro/utility_macros.xacro (robot description, xacro)
@@ -66,4 +66,5 @@
       <origin xyz="${x} ${y} ${z}" rpy="${-pi/2} 0 0" />
       <axis xyz="0 0 1" />
+      <limit effort="30.0" velocity="10.0"/> <!-- 10 rad/s ~ 2.5 mph top speed assuming 9 in diameter tires-->
     </joint>
   </xacro:macro>

File: src/uirover_hardware/xacro/ros2_control.urdf.xacro (robot description, xacro)
@@ -4,15 +4,4 @@
     <xacro:arg name="hw_type" default="target"/>
     <xacro:property name='hw_type' value="$(arg hw_type)"/>
-    <gazebo>
-        <plugin filename="gz_ros2_control-system" name="gz_ros2_control::GazeboSimROS2ControlPlugin">
-            <ros>
-                <namespace>/uirover/control</namespace>
-            </ros>
-            <parameters>$(find uirover_controllers)/config/controllers.yaml</parameters>
-        </plugin>
-        <plugin filename="gz-sim-sensors-system" name="gz::sim::systems::Sensors">
-            <render_engine>ogre2</render_engine>
-        </plugin>
-    </gazebo>
     <ros2_control name="wheels_hardware" type="system">
         <hardware>
