Commit message: updated moveit config, missing deps, changed wheels to fixed joint because of moveit2 weirdness

File: src/uirover_description/xacro/utility_macros.xacro (robot description, xacro)
@@ -61,9 +61,9 @@
         length="${wheel_width}" />
     </link>
-    <joint name="${name}_joint" type="continuous">
+    <joint name="${name}_joint" type="fixed">
       <parent link="${parent}" />
       <child link="${name}" />
       <origin xyz="${x} ${y} ${z}" rpy="${-pi/2} 0 0" />
-      <axis xyz="0 0 1" />
+      <!-- <axis xyz="0 0 1" /> -->
     </joint>
   </xacro:macro>

File: src/uirover_moveit/config/uirover.urdf.xacro (robot description, xacro)
@@ -3,5 +3,5 @@
     <xacro:arg name="initial_positions_file" default="initial_positions.yaml" />
     <!-- Import uirover urdf file -->
-    <xacro:include filename="$(find uirover_description)/xacro/arm.urdf.xacro" />
+    <xacro:include filename="$(find uirover_description)/urdf/uirover.urdf.xacro" />
     <!-- Import control_xacro -->
     <xacro:include filename="uirover.ros2_control.xacro" />
