Commit message: minor urdf tweaks

File: src/uirover_description/xacro/arm.urdf.xacro (robot description, xacro)
@@ -5,4 +5,9 @@
     </material>
     <link name="arm_base_link"></link>
+    <joint name="arm_base_joint" type="fixed">
+        <parent link="base_link" />
+        <child link="arm_base_link" />
+        <origin xyz="0.2 0 0" rpy="0 0 0" />
+    </joint>
     <link name="arm_l0">
         <visual>
@@ -158,14 +163,14 @@
         <visual>
             <geometry>
-                <box size=".1 .1 .1"/>
+                <box size=".02 .02 .1"/>
             </geometry>
-            <origin xyz="0 0 0.05" rpy="0 0 0" />
+            <origin xyz="0 0 -0.05" rpy="0 0 0" />
             <material name="grey"/>
         </visual>
         <collision>
             <geometry>
-                <box size=".1 .1 .1"/>
+                <box size=".02 .02 .1"/>
             </geometry>
-            <origin xyz="0 0 0.05" rpy="0 0 0" />
+            <origin xyz="0 0 -0.05" rpy="0 0 0" />
         </collision>
     </link>
@@ -173,5 +178,5 @@
         <parent link="arm_l5" />
         <child link="end_effector" />
-        <origin xyz="0 0 0.05" rpy="0 0 0" />
+        <origin xyz="0 0 0.12" rpy="0 0 0" />
     </joint>
 </robot>

Commit message: gazebo, mock hardware, and target configurations now all use same urdf and launch file

File: src/uirover_description/xacro/arm.urdf.xacro (robot description, xacro)
@@ -35,5 +35,5 @@
         <origin xyz="0 0 0" rpy="0 0 0" />
         <axis xyz="0 0 1" />
-        <limit lower="-2.0" upper="2.0" effort="10.0" velocity="0.5"/>
+        <limit lower="-3.0" upper="3.0" effort="40.0" velocity="0.5"/>
     </joint>
     <link name="arm_l1">
@@ -68,5 +68,5 @@
         <origin xyz="0 0 0.104" rpy="0 0 0" />
         <axis xyz="0 1 0" />
-        <limit lower="-2.0" upper="2.0" effort="10.0" velocity="0.5"/>
+        <limit lower="-3.0" upper="3.0" effort="40.0" velocity="0.5"/>
     </joint>
     <link name="arm_l2">
@@ -101,5 +101,5 @@
         <origin xyz="0 0 0.534" rpy="0 0 0" />
         <axis xyz="0 1 0" />
-        <limit lower="-${pi}" upper="${pi}" effort="10.0" velocity="0.5"/>
+        <limit lower="-${pi}" upper="${pi}" effort="40.0" velocity="0.5"/>S
     </joint>
     <link name="arm_l3">
@@ -140,5 +140,5 @@
         <origin xyz="0 0.076 0.203" rpy="0 0 0" />
         <axis xyz="1 0 0" />
-        <limit lower="${-pi}" upper="${pi}" effort="10.0" velocity="0.5"/>
+        <limit lower="${-pi}" upper="${pi}" effort="40.0" velocity="0.5"/>
     </joint>
     <link name="arm_l4">
@@ -167,5 +167,5 @@
         <origin xyz="0 -0.025 0.179" rpy="0 0 0" />
         <axis xyz="0 1 0" />
-        <limit lower="${-pi}" upper="${pi}" effort="10.0" velocity="0.5"/>
+        <limit lower="${-pi}" upper="${pi}" effort="40.0" velocity="0.5"/>
     </joint>
     <link name="arm_l5">
@@ -194,5 +194,5 @@
         <origin xyz="0 -0.075 0.08" rpy="0 0 0" />
         <axis xyz="0 0 1" />
-        <limit effort="10.0" velocity="0.5"/>
+        <limit effort="40.0" velocity="0.5"/>
     </joint>
     <link name="end_effector">
