Commit message: Enhance navigation and perception capabilities; added EKF configuration, integrated GPS and depth camera sensors, and updated launch files for improved simulation support.

File: src/uirover_description/xacro/gazebo.urdf.xacro (robot description, xacro)
@@ -12,5 +12,5 @@
             <render_engine>ogre2</render_engine>
         </plugin>
-        <plugin filename="gz-sim-sensors-navsat" name="gz::sim::systems::NavSat">
+        <plugin filename="gz-sim-navsat-system" name="gz::sim::systems::NavSat">
         </plugin>
     </gazebo>

File: src/uirover_description/xacro/sensors.urdf.xacro (robot description, xacro)
@@ -3,4 +3,5 @@
     xmlns:xacro="http://www.ros.org/wiki/xacro">
     <xacro:include filename="$(find uirover_description)/xacro/utility_macros.xacro" />
+    <!-- http://sdformat.org/spec?ver=1.9&elem=sensor -->
     <xacro:macro name="arducam" params="name">
         <link name="${name}">
@@ -53,50 +54,141 @@
     <!-- =============================== -->
     <!-- ARDUCAM CAMERA -->
-    <xacro:arducam name="antenna_camera" />
+    <!-- <xacro:arducam name="antenna_camera" />
     <joint name="antenna_camera_joint" type="fixed">
         <origin xyz="-0.24 0.28 1.3" rpy="0.0 0.5 0.0" />
         <parent link="base_link" />
         <child link="antenna_camera" />
-    </joint>
-    <link name="ZED_F9P_GPS">
-        <gazebo reference="ZED_F9P_GPS">
-            <sensor name="ZED_F9P_GPS" type="navsat">
-                <navsat>
-                    <position_sensing>
-                        <horizontal>
-                            <noise type="gaussian">
-                                <mean>0</mean>
-                                <stddev>1.75e-6</stddev>
-                            </noise>
-                        </horizontal>
-                        <vertical>
-                            <noise type="gaussian">
-                                <mean>0.0</mean>
-                                <stddev>1.35e-6</stddev>
-                            </noise>
-                        </vertical>
-                    </position_sensing>
-                    <vertical_sensing>
-                        <horizontal>
-                            <noise type="gaussian">
-                                <mean>0.0</mean>
-                                <stddev>0.0001</stddev>
-                            </noise>
-                        </horizontal>
-                        <vertical>
-                            <noise type="gaussian">
-                                <mean>0.0</mean>
-                                <stddev>0.0001</stddev>
-                            </noise>
-                        </vertical>
-                    </vertical_sensing>
-                </navsat>
-            </sensor>
-        </gazebo>
-    </link>
-    <joint name="ZED_F9P_GPS_joint" type="fixed">
+    </joint> -->
+    <link name="zed_f9p_gps"></link>
+    <gazebo reference="zed_f9p_gps">
+        <sensor name="zed_f9p_gps" type="navsat">
+            <topic>navsat</topic>
+            <always_on>true</always_on>
+            <update_rate>10</update_rate>
+            <navsat>
+                <!-- <position_sensing>
+                    <horizontal>
+                        <noise type="gaussian">
+                            <mean>0</mean>
+                            <stddev>1.75e-6</stddev>
+                        </noise>
+                    </horizontal>
+                    <vertical>
+                        <noise type="gaussian">
+                            <mean>0.0</mean>
+                            <stddev>1.35e-6</stddev>
+                        </noise>
+                    </vertical>
+                </position_sensing> -->
+            </navsat>
+        </sensor>
+    </gazebo>
+    <joint name="zed_f9p_gps_joint" type="fixed">
+        <!-- TODO origin coords are a placeholder. not important unless using RTK -->
         <origin xyz="0 0 0"/>
         <parent link="base_link"/>
-        <child link="ZED_F9P_GPS"/>
+        <child link="zed_f9p_gps"/>
+    </joint>
+    <!-- https://cdrdv2-public.intel.com/841984/Intel-RealSense-D400-Series-Datasheet.pdf -->
+    <link name="d435i_depth_cam"></link>
+    <gazebo reference="d435i_depth_cam">
+        <sensor name="d435i_depth_cam" type="depth">
+            <topic>/d435i_rgbd</topic>
+            <always_on>1</always_on>
+            <update_rate>10</update_rate>
+            <visualize>true</visualize>
+            <camera>
+                <!-- 86 deg FOV -->
+                <camera_info_topic>/d435i_rgbd_info</camera_info_topic>
+                <optical_frame_id>d435i_depth_cam</optical_frame_id>
+                <horizontal_fov>1.50098</horizontal_fov>
+                <image>
+                    <!-- Low resolution for performance reasons -->
+                    <width>640</width>
+                    <height>380</height>
+                    <format>B8G8R8</format>
+                </image>
+                <clip>
+                    <near>0.01</near>
+                    <far>5</far>                    <!-- required unless youre using a NASA super computer-->
+                </clip>
+                <depth_camera>
+                    <output>depths</output>
+                </depth_camera>
+            </camera>
+        </sensor>
+    </gazebo>
+    <joint name="d435i_depth_cam_joint" type="fixed">
+        <!-- TODO origin coords are a placeholder. not important unless using RTK -->
+        <origin xyz="0.4 0.2 0"/>
+        <parent link="base_link"/>
+        <child link="d435i_depth_cam"/>
+    </joint>
+    <link name="imu_link"></link>
+    <sensor name="imu_sensor" type="imu">
+        <always_on>true</always_on>
+        <update_rate>100</update_rate>
+        <visualize>true</visualize>
+        <topic>/imu</topic>
+        <!-- <gz_frame_id>imu_link</gz_frame_id> -->
+        <imu>
+            <angular_velocity>
+                <x>
+                    <noise type="gaussian">
+                        <mean>0.0</mean>
+                        <stddev>2e-4</stddev>
+                        <bias_mean>0.0000075</bias_mean>
+                        <bias_stddev>0.0000008</bias_stddev>
+                    </noise>
+                </x>
+                <y>
+                    <noise type="gaussian">
+                        <mean>0.0</mean>
+                        <stddev>2e-4</stddev>
+                        <bias_mean>0.0000075</bias_mean>
+                        <bias_stddev>0.0000008</bias_stddev>
+                    </noise>
+                </y>
+                <z>
+                    <noise type="gaussian">
+                        <mean>0.0</mean>
+                        <stddev>2e-4</stddev>
+                        <bias_mean>0.0000075</bias_mean>
+                        <bias_stddev>0.0000008</bias_stddev>
+                    </noise>
+                </z>
+            </angular_velocity>
+            <linear_acceleration>
+                <x>
+                    <noise type="gaussian">
+                        <mean>0.0</mean>
+                        <stddev>1.7e-2</stddev>
+                        <bias_mean>0.1</bias_mean>
+                        <bias_stddev>0.001</bias_stddev>
+                    </noise>
+                </x>
+                <y>
+                    <noise type="gaussian">
+                        <mean>0.0</mean>
+                        <stddev>1.7e-2</stddev>
+                        <bias_mean>0.1</bias_mean>
+                        <bias_stddev>0.001</bias_stddev>
+                    </noise>
+                </y>
+                <z>
+                    <noise type="gaussian">
+                        <mean>0.0</mean>
+                        <stddev>1.7e-2</stddev>
+                        <bias_mean>0.1</bias_mean>
+                        <bias_stddev>0.001</bias_stddev>
+                    </noise>
+                </z>
+            </linear_acceleration>
+        </imu>
+    </sensor>
+    <joint name="imu_sensor_joint" type="fixed">
+        <origin xyz="0 0 0"/>
+        <parent link="base_link"/>
+        <child link="imu_link"/>
     </joint>
 </robot>

Commit message: work on robot localization via EKF

File: src/uirover_description/xacro/gazebo.urdf.xacro (robot description, xacro)
@@ -12,6 +12,6 @@
             <render_engine>ogre2</render_engine>
         </plugin>
-        <plugin filename="gz-sim-navsat-system" name="gz::sim::systems::NavSat">
-        </plugin>
+        <plugin filename="gz-sim-navsat-system" name="gz::sim::systems::NavSat"></plugin>
+        <plugin filename="gz-sim-imu-system" name="gz::sim::systems::Imu"></plugin>
     </gazebo>
 </robot>

File: src/uirover_description/xacro/sensors.urdf.xacro (robot description, xacro)
@@ -45,5 +45,5 @@
                 </camera>
                 <always_on>1</always_on>
-                <update_rate>30</update_rate>
+                <update_rate>5</update_rate>
                 <visualize>true</visualize>
             </sensor>
@@ -54,10 +54,10 @@
     <!-- =============================== -->
     <!-- ARDUCAM CAMERA -->
-    <!-- <xacro:arducam name="antenna_camera" />
+    <xacro:arducam name="antenna_camera" />
     <joint name="antenna_camera_joint" type="fixed">
         <origin xyz="-0.24 0.28 1.3" rpy="0.0 0.5 0.0" />
         <parent link="base_link" />
         <child link="antenna_camera" />
-    </joint> -->
+    </joint>
     <link name="zed_f9p_gps"></link>
     <gazebo reference="zed_f9p_gps">
@@ -65,5 +65,5 @@
             <topic>navsat</topic>
             <always_on>true</always_on>
-            <update_rate>10</update_rate>
+            <update_rate>5</update_rate>
             <navsat>
                 <!-- <position_sensing>
@@ -96,5 +96,5 @@
             <topic>/d435i_rgbd</topic>
             <always_on>1</always_on>
-            <update_rate>10</update_rate>
+            <update_rate>5</update_rate>
             <visualize>true</visualize>
             <camera>
@@ -125,70 +125,72 @@
         <child link="d435i_depth_cam"/>
     </joint>
-    <link name="imu_link"></link>
-    <sensor name="imu_sensor" type="imu">
-        <always_on>true</always_on>
-        <update_rate>100</update_rate>
-        <visualize>true</visualize>
-        <topic>/imu</topic>
-        <!-- <gz_frame_id>imu_link</gz_frame_id> -->
-        <imu>
-            <angular_velocity>
-                <x>
-                    <noise type="gaussian">
-                        <mean>0.0</mean>
-                        <stddev>2e-4</stddev>
-                        <bias_mean>0.0000075</bias_mean>
-                        <bias_stddev>0.0000008</bias_stddev>
-                    </noise>
-                </x>
-                <y>
-                    <noise type="gaussian">
-                        <mean>0.0</mean>
-                        <stddev>2e-4</stddev>
-                        <bias_mean>0.0000075</bias_mean>
-                        <bias_stddev>0.0000008</bias_stddev>
-                    </noise>
-                </y>
-                <z>
-                    <noise type="gaussian">
-                        <mean>0.0</mean>
-                        <stddev>2e-4</stddev>
-                        <bias_mean>0.0000075</bias_mean>
-                        <bias_stddev>0.0000008</bias_stddev>
-                    </noise>
-                </z>
-            </angular_velocity>
-            <linear_acceleration>
-                <x>
-                    <noise type="gaussian">
-                        <mean>0.0</mean>
-                        <stddev>1.7e-2</stddev>
-                        <bias_mean>0.1</bias_mean>
-                        <bias_stddev>0.001</bias_stddev>
-                    </noise>
-                </x>
-                <y>
-                    <noise type="gaussian">
-                        <mean>0.0</mean>
-                        <stddev>1.7e-2</stddev>
-                        <bias_mean>0.1</bias_mean>
-                        <bias_stddev>0.001</bias_stddev>
-                    </noise>
-                </y>
-                <z>
-                    <noise type="gaussian">
-                        <mean>0.0</mean>
-                        <stddev>1.7e-2</stddev>
-                        <bias_mean>0.1</bias_mean>
-                        <bias_stddev>0.001</bias_stddev>
-                    </noise>
-                </z>
-            </linear_acceleration>
-        </imu>
-    </sensor>
+    <link name="imu_sensor"></link>
+    <gazebo reference="imu_sensor">
+        <sensor name="imu_sensor" type="imu">
+            <always_on>true</always_on>
+            <update_rate>5</update_rate>
+            <visualize>true</visualize>
+            <topic>/imu</topic>
+            <imu>
+                <enable_orientation>true</enable_orientation>
+                <angular_velocity>
+                    <x>
+                        <noise type="gaussian">
+                            <mean>0.0</mean>
+                            <stddev>2e-4</stddev>
+                            <bias_mean>0.0000075</bias_mean>
+                            <bias_stddev>0.0000008</bias_stddev>
+                        </noise>
+                    </x>
+                    <y>
+                        <noise type="gaussian">
+                            <mean>0.0</mean>
+                            <stddev>2e-4</stddev>
+                            <bias_mean>0.0000075</bias_mean>
+                            <bias_stddev>0.0000008</bias_stddev>
+                        </noise>
+                    </y>
+                    <z>
+                        <noise type="gaussian">
+                            <mean>0.0</mean>
+                            <stddev>2e-4</stddev>
+                            <bias_mean>0.0000075</bias_mean>
+                            <bias_stddev>0.0000008</bias_stddev>
+                        </noise>
+                    </z>
+                </angular_velocity>
+                <linear_acceleration>
+                    <x>
+                        <noise type="gaussian">
+                            <mean>0.0</mean>
+                            <stddev>1.7e-2</stddev>
+                            <bias_mean>0.1</bias_mean>
+                            <bias_stddev>0.001</bias_stddev>
+                        </noise>
+                    </x>
+                    <y>
+                        <noise type="gaussian">
+                            <mean>0.0</mean>
+                            <stddev>1.7e-2</stddev>
+                            <bias_mean>0.1</bias_mean>
+                            <bias_stddev>0.001</bias_stddev>
+                        </noise>
+                    </y>
+                    <z>
+                        <noise type="gaussian">
+                            <mean>0.0</mean>
+                            <stddev>1.7e-2</stddev>
+                            <bias_mean>0.1</bias_mean>
+                            <bias_stddev>0.001</bias_stddev>
+                        </noise>
+                    </z>
+                </linear_acceleration>
+            </imu>
+        </sensor>
+    </gazebo>
     <joint name="imu_sensor_joint" type="fixed">
         <origin xyz="0 0 0"/>
         <parent link="base_link"/>
-        <child link="imu_link"/>
+        <child link="imu_sensor"/>
     </joint>
 </robot>

File: src/uirover_hardware/xacro/ros2_control.urdf.xacro (robot description, xacro)
@@ -129,3 +129,18 @@
         </joint>
     </ros2_control>
+    <ros2_control name="imu_sensor_system" type="sensor">
+        <!-- IMU Sensor Definition -->
+        <sensor name="imu_sensor">
+            <state_interface name="orientation.x"/>
+            <state_interface name="orientation.y"/>
+            <state_interface name="orientation.z"/>
+            <state_interface name="orientation.w"/>
+            <state_interface name="angular_velocity.x"/>
+            <state_interface name="angular_velocity.y"/>
+            <state_interface name="angular_velocity.z"/>
+            <state_interface name="linear_acceleration.x"/>
+            <state_interface name="linear_acceleration.y"/>
+            <state_interface name="linear_acceleration.z"/>
+        </sensor>
+    </ros2_control>
 </robot>
